File: hardware/ffp5cs-wroom-prod-230v/kicad/ffp5cs-wroom-prod-230v.kicad_sch (KiCad schematic)
At the start: 70 parts, among them J1 Bornier_5.08, J10 JST-XH, J11 Bornier_5.08, J12 Bornier_5.08, J13 Support OLED, J14 Support I2C ext, J15 Header servo, J16 Header servo, J17 Header GPIO libres, J18 Bornier_5.08, J19 Bornier_5.08, J2 Jack 5.5/2.1, J20 Header alim, J3 Bornier_5.08, J4 Bornier_5.08, J5 Bornier_5.08, J6 Bornier_5.08, J7 JST-XH, J8 JST-XH, J9 JST-XH, K1 SRD-05VDC-SL-C, K2 SRD-05VDC-SL-C, K3 SRD-05VDC-SL-C, K4 SRD-05VDC-SL-C, Q1 BC337-40, Q2 BC337-40, Q3 BC337-40, Q4 BC337-40

Commit message: hardware(ffp5cs): 3 ports I2C libres par carte + pipeline de routage LV scripté
Demande : pouvoir brancher des modules I2C supplémentaires sans soudure.
Avec les pull-ups 4.7k en place, 3-4 modules simultanés sont confortables
(limite = capacité du bus, pas l'ESP) — dimensionné en conséquence :

- 12/24V (rev 0.4) : +J18 +J19 (supports 1x4 GND/VCC/SCL/SDA, mêmes nets
  que J14) ; netclasses Relais/Alim désormais émises par generate.py ;
  nouveau generator/route_lv.py (pipeline scripté dérivé de route_230v.py :
  freerouting, vias de couture, îlots supprimés, reliefs corrigés, bandes
  de bord) ; re-routage complet, gerbers v0.4 (remplacent v0.3).
- 230V (rev 0.2) : +J21 +J22 idem ; bandes de keepout le long des bords
  ajoutées au pipeline (l'autorouteur frôlait l'edge clearance) ;
  re-routage complet, gerbers v0.2 (remplacent v0.1).
- Validation des DEUX cartes : ERC 0 erreur, DRC 0 violation, 0 pad non
  connecté, contrôle 3mm secteur/logique (230V) : 0 écart, checker
  pins.h <-> schéma <-> PCB vert.
- READMEs : ports I2C documentés (3-4 modules max, bus < ~50cm, sinon
  pull-ups 2.2k).

Co-Authored-By: Claude Fable 5 <noreply@anthropic.com>
Claude-Session: https://claude.ai/code/session_01HcxShQb65yktRwp31wBq9q
Parts:
- added J21, J22: Support I2C libre, ffp5cs:PinSocket_1x04_P2.54mm_Vertical, symbol ffp5cs:CONN_04
Connections:
- net +3V3: now also J21.2, J22.2
- net GND: now also J21.1, J22.1
- net I2C_SCL_GPIO22: now also J21.3, J22.3
- net I2C_SDA_GPIO21: now also J21.4, J22.4
Changed lines of the file:
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@@
     (title "ffp5cs wroom-prod - carte porteuse ESP32 DevKit V1")
     (date "2026-07-07")
-    (rev "0.1")
+    (rev "0.2")
     (company "salle aeree n3")
     (comment 1 "Genere par hardware/ffp5cs-wroom-prod/generator/generate.py")
@@
     (effects (font (size 1.27 1.27)) (justify left bottom))
 )
+  (symbol (lib_id "ffp5cs:CONN_04") (at 264.16 254.00 0) (unit 1)
+    (exclude_from_sim no) (in_bom yes) (on_board yes) (dnp no)
+    (property "Reference" "J21" (at 264.16 243.84 0) (effects (font (size 1.27 1.27))))
+    (property "Value" "Support I2C libre" (at 264.16 245.98 0) (effects (font (size 1.27 1.27))))
+    (property "Footprint" "ffp5cs:PinSocket_1x04_P2.54mm_Vertical" (at 264.16 254.00 0) (effects (font (size 1.27 1.27)) (hide yes)))
+    (property "Datasheet" "~" (at 264.16 254.00 0) (effects (font (size 1.27 1.27)) (hide yes)))
+    (property "Description" "Port I2C libre 2 (1=GND 2=VCC 3=SCL 4=SDA)" (at 264.16 254.00 0) (effects (font (size 1.27 1.27)) (hide yes)))
+    (pin "1")
+    (pin "2")
+    (pin "3")
+    (pin "4")
+    (instances (project "ffp5cs-wroom-prod-230v" (path "/bdc3ceab-d5f3-5c3a-89af-564c4cb456f7" (reference "J21") (unit 1))))
+  )
+  (wire (pts (xy 257.81 248.92) (xy 255.27 248.92))
+    (stroke (width 0) (type default)))
+  (label "GND" (at 255.27 248.92 0)
+    (effects (font (size 1.27 1.27)) (justify right bottom))
+)
+  (wire (pts (xy 257.81 251.46) (xy 255.27 251.46))
+    (stroke (width 0) (type default)))
+  (label "+3V3" (at 255.27 251.46 0)
+    (effects (font (size 1.27 1.27)) (justify right bottom))
+)
+  (wire (pts (xy 257.81 254.00) (xy 255.27 254.00))
+    (stroke (width 0) (type default)))
+  (label "I2C_SCL_GPIO22" (at 255.27 254.00 0)
+    (effects (font (size 1.27 1.27)) (justify right bottom))
+)
+  (wire (pts (xy 257.81 256.54) (xy 255.27 256.54))
+    (stroke (width 0) (type default)))
+  (label "I2C_SDA_GPIO21" (at 255.27 256.54 0)
+    (effects (font (size 1.27 1.27)) (justify right bottom))
+)
+  (symbol (lib_id "ffp5cs:CONN_04") (at 264.16 274.32 0) (unit 1)
+    (exclude_from_sim no) (in_bom yes) (on_board yes) (dnp no)
+    (property "Reference" "J22" (at 264.16 264.16 0) (effects (font (size 1.27 1.27))))
+    (property "Value" "Support I2C libre" (at 264.16 266.30 0) (effects (font (size 1.27 1.27))))
+    (property "Footprint" "ffp5cs:PinSocket_1x04_P2.54mm_Vertical" (at 264.16 274.32 0) (effects (font (size 1.27 1.27)) (hide yes)))
+    (property "Datasheet" "~" (at 264.16 274.32 0) (effects (font (size 1.27 1.27)) (hide yes)))
+    (property "Description" "Port I2C libre 3 (1=GND 2=VCC 3=SCL 4=SDA)" (at 264.16 274.32 0) (effects (font (size 1.27 1.27)) (hide yes)))
+    (pin "1")
+    (pin "2")
+    (pin "3")
+    (pin "4")
+    (instances (project "ffp5cs-wroom-prod-230v" (path "/bdc3ceab-d5f3-5c3a-89af-564c4cb456f7" (reference "J22") (unit 1))))
+  )
+  (wire (pts (xy 257.81 269.24) (xy 255.27 269.24))
+    (stroke (width 0) (type default)))
+  (label "GND" (at 255.27 269.24 0)
+    (effects (font (size 1.27 1.27)) (justify right bottom))
+)
+  (wire (pts (xy 257.81 271.78) (xy 255.27 271.78))
+    (stroke (width 0) (type default)))
+  (label "+3V3" (at 255.27 271.78 0)
+    (effects (font (size 1.27 1.27)) (justify right bottom))
+)
+  (wire (pts (xy 257.81 274.32) (xy 255.27 274.32))
+    (stroke (width 0) (type default)))
+  (label "I2C_SCL_GPIO22" (at 255.27 274.32 0)
+    (effects (font (size 1.27 1.27)) (justify right bottom))
+)
+  (wire (pts (xy 257.81 276.86) (xy 255.27 276.86))
+    (stroke (width 0) (type default)))
+  (label "I2C_SDA_GPIO21" (at 255.27 276.86 0)
+    (effects (font (size 1.27 1.27)) (justify right bottom))
+)
   (symbol (lib_id "ffp5cs:CONN_14") (at 60.96 177.80 0) (unit 1)

Commit message: feat(ffp5cs+hardware): relais AUX1/AUX2 (firmware v15.26, carte 230V 6 canaux) + corrections des 2 cartes
FIRMWARE ffp5cs v15.26 :
- Pins::AUX1/AUX2 (WROOM 23/25, S3 47/48), RelayController generique,
  SystemActuators::setAux/isAuxOn, IActuators::setAux (defaut no-op,
  doubles de test intacts), GPIOMap::AUX1/AUX2 dans ALL_MAPPINGS
  (parser GET + NVS + restauration boot automatiques).
- Garde test_mapping_count_is_stable 27->29 (ajout conscient).
- Tests natifs : 54 suites PASSED ; build wroom-test SUCCESS
  (wroom-prod local refuse par design les secrets placeholder).
- Contrat POST inchange ; cote serveur : n3_serveur 6.38.0 (PR jumelle).

HARDWARE 230V rev 0.3 — 6 canaux (234x110mm) :
- +REL5/REL6 (AUX1/AUX2) : relais+bornier+fentes identiques aux 4 canaux
  metier, refs dediees (R28-R33, D6/D7, LED6/LED7, Q5/Q6, J23/J24).
- J17 breakout 1x14 -> 1x12 (IO23/IO25 ne sont plus des spares).
- Pipeline : bande secteur etendue, min via 0.5, jar freerouting 2.x,
  timeout 1500s. Valide : ERC 0, DRC 0 violation 0 non-connecte,
  controle 3mm secteur/logique 0 ecart, checker 16 signaux vert.
- Gerbers v0.3, fritzing 6 commandes relais, README.

CORRECTIONS COMMUNES (12/24V rev 0.5 + 230V) :
- BOM : ligne 'A1 (supports)' (2 barrettes femelles 1x15) — le DevKit
  est enfichable, jamais soude, mais les supports n'etaient pas commandables.
- Keepout cuivre sous l'antenne WiFi du module (2 faces) + note serigraphiee
  deplacee cote antenne (elle etait sous le corps du module, cote USB).
- Checker etendu a la topologie des canaux HC-SR04 (JST 1=+5V 2=GPIO
  3=ECHO 4=GND ; 1k serie echo ; 2k pull-down) sur les deux cartes.
- 12/24V : pinmap declare AUX1/AUX2 -> spares J17 (modules relais externes) ;
  re-route complet (jar 1.9, le 2.1 depassait le timeout sur cette carte),
  DRC 0/0, gerbers v0.5.

Co-Authored-By: Claude Fable 5 <noreply@anthropic.com>
Claude-Session: https://claude.ai/code/session_01HcxShQb65yktRwp31wBq9q
Parts:
- added D6, D7: 1N4007, ffp5cs:D_DO-41_SOD81_P10.16mm_Horizontal, symbol ffp5cs:D
- added J23, J24: Bornier_5.08, ffp5cs:TerminalBlock_bornier-3_P5.08mm, symbol ffp5cs:CONN_03
- added K5, K6: SRD-05VDC-SL-C, ffp5cs:Relay_SPDT_SANYOU_SRD_Series_Form_C, symbol ffp5cs:RELAY_SRD
- added LED6, LED7: rouge, ffp5cs:LED_D5.0mm, symbol ffp5cs:LED
- added Q5, Q6: BC337-40, ffp5cs:TO-92_Inline, symbol ffp5cs:NPN
- added R28, R30, R31, R33: 1k, ffp5cs:R_Axial_DIN0207_L6.3mm_D2.5mm_P10.16mm_Horizontal, symbol ffp5cs:R
- added R29, R32: 10k, ffp5cs:R_Axial_DIN0207_L6.3mm_D2.5mm_P10.16mm_Horizontal, symbol ffp5cs:R
- J17: footprint ffp5cs:PinHeader_1x14_P2.54mm_Vertical -> ffp5cs:PinHeader_1x12_P2.54mm_Vertical; symbol ffp5cs:CONN_14 -> ffp5cs:CONN_12
Connections:
- net +5V: now also D6.1 (K), D7.1 (K), K5.5 (COIL+), K6.5 (COIL+), R30.1, R33.1
- net GND: now also Q5.3 (E), Q6.3 (E), R29.2, R32.2
- net SPARE_GPIO32: now also J17.9; no longer J17.11
- net SPARE_GPIO35: now also J17.10; no longer J17.12
- net SPARE_GPIO36: now also J17.11; no longer J17.13
- net SPARE_GPIO39: now also J17.12; no longer J17.14
- net SPARE_GPIO23 renamed AUX1_GPIO23
- net AUX1_GPIO23: now also R28.1; no longer J17.9
- net SPARE_GPIO25 renamed AUX2_GPIO25
- net AUX2_GPIO25: now also R31.1; no longer J17.10
- new net REL5_B: Q5.2 (B), R28.2, R29.1
- new net REL5_COM: J23.2, K5.1 (COM)
- new net REL5_LED: LED6.2 (A), R30.2
- new net REL5_NC: J23.1, K5.4 (NC)
- new net REL5_NO: J23.3, K5.3 (NO)
- new net REL5_SW: D6.2 (A), K5.2 (COIL-), LED6.1 (K), Q5.1 (C)
- new net REL6_B: Q6.2 (B), R31.2, R32.1
- new net REL6_COM: J24.2, K6.1 (COM)
- new net REL6_LED: LED7.2 (A), R33.2
- new net REL6_NC: J24.1, K6.4 (NC)
- new net REL6_NO: J24.3, K6.3 (NO)
- new net REL6_SW: D7.2 (A), K6.2 (COIL-), LED7.1 (K), Q6.1 (C)
