File: hardware/n3pp-msp-commun/kicad/n3pp-msp-commun.kicad_pcb (KiCad board)
At the start: 2 copper layers, 210 x 105 mm, 98 parts, among them J1 Bornier_5.08, J10 JST-XH, J11 JST-XH, J12 Bornier_5.08, J13 JST-XH, J14 Support OLED, J15 Support I2C libre, J16 Support I2C libre, J17 Support I2C libre, J18 Header GPIO libres, J19 Rail alim Dupont, J2 Jack 5.5/2.1, J20 Header servo, J21 Header servo, J22 Bornier_5.08, J23 Bornier_5.08, J24 Bornier_5.08, J25 Bornier_5.08, J26 Bornier_5.08, J27 Bornier_5.08, J28 Bornier_5.08, J29 Bornier_5.08, J3 Bornier_5.08, J4 Bornier_5.08, J5 Bornier_5.08, J6 Bornier_5.08, J7 Bornier_5.08, J8 Bornier_5.08, J9 JST-XH, K1 SRD-05VDC-SL-C, K2 SRD-05VDC-SL-C, K3 SRD-05VDC-SL-C, K4 SRD-05VDC-SL-C, K5 SRD-05VDC-SL-C, K6 SRD-05VDC-SL-C, Q1 BC337-40, Q2 BC337-40, Q3 BC337-40, Q4 BC337-40, Q5 BC337-40, Q6 BC337-40

Commit message: fix(hardware): fichiers de fabrication et sérigraphie prêts pour JLCPCB
Trois défauts trouvés en préparant une commande, sur les 3 cartes :

1. Sérigraphie sous les minima fabricant : textes de 0,8 mm de haut / 0,12 mm
   de trait, alors que JLCPCB exige 1 mm / 0,15 mm — les étiquettes de câblage
   (NO COM NC, ADC A 33, ZONE 230V - DANGER...) risquaient d'être floutées ou
   supprimées par leur DFM. Tous les textes passent à >= 1 mm / 0,16 mm.
2. Repères de composants superposés aux étiquettes (34 chevauchements, dont
   l'avertissement 230 V masqué par K3/K4). Nouveau generator/tidy_silkscreen.py :
   écarte le repère (court, recasable) sans jamais bouger l'étiquette dont la
   position porte le sens. Déterministe, idempotent, avec audit final par couche.
   Titre de la carte 12/24 V déplacé (il croisait REL2/REL3).
3. Zip Gerbers de la carte commune pollué par 6 couches de documentation
   (F.Fab, *.Courtyard, User.*, Margin) et perçages PTH/NPTH fusionnés.
   Nouveau generator/export_fab.py : exactement les 7 couches utiles + PTH/NPTH
   séparés (trous M3 non métallisés) + rendus de revue sans cartouche de page.
   Aucun script d'export n'existait dans le dépôt — les exports n'étaient pas
   reproductibles, d'où la divergence entre cartes.

Ajouts : marqueur JLCJLCJLCJLC au dos des 3 cartes (emplacement du numéro de
commande imposé au fabricant, gratuit, plutôt qu'au hasard sur une étiquette),
et hardware/COMMANDE_JLCPCB.md — réglages du formulaire expliqués un par un,
choix par carte (1 oz vs 2 oz pour le 230 V, confirmation des fentes fraisées).

Cuivre inchangé : DRC 0 violation / 0 pastille non connectée sur les 3 cartes,
règle .kicad_dru 3 mm secteur toujours vérifiée sur la carte 230 V.

Co-Authored-By: Claude Opus 5 <noreply@anthropic.com>
Claude-Session: https://claude.ai/code/session_01HcxShQb65yktRwp31wBq9q
Other:
- board text added: "JLCJLCJLCJLC"
Changed lines of the file:
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@@
 		(tags "connector JST XH vertical")
 		(property "Reference" "J11"
-			(at 2.5 -3.55 0)
+			(at 2.5 -2.55 0)
 			(layer "F.SilkS")
 			(effects
@@
 		(tags "connector JST XH vertical")
 		(property "Reference" "J10"
-			(at 2.5 -3.55 0)
+			(at 2.5 -2.55 0)
 			(layer "F.SilkS")
 			(effects
@@
 		(tags "terminal block bornier3")
 		(property "Reference" "J6"
-			(at 5.05 -4.65 0)
+			(at 5.05 -6.65 0)
 			(layer "F.SilkS")
 			(effects
@@
 		(tags "terminal block bornier3")
 		(property "Reference" "J7"
-			(at 5.05 -4.65 0)
+			(at 5.05 -6.65 0)
 			(layer "F.SilkS")
 			(effects
@@
 		(tags "Through hole pin header THT 1x07 2.54mm single row")
 		(property "Reference" "J18"
-			(at 0 -2.33 0)
+			(at 0 -3.33 0)
 			(layer "F.SilkS")
 			(effects
@@
 		(tags "connector JST XH vertical")
 		(property "Reference" "J9"
-			(at 2.5 -3.55 0)
+			(at 2.5 -2.55 0)
 			(layer "F.SilkS")
 			(effects
@@
 		(tags "terminal block bornier3")
 		(property "Reference" "J5"
-			(at 5.05 -4.65 0)
+			(at 5.05 -6.65 0)
 			(layer "F.SilkS")
 			(effects
@@
 		(tags "ESP32 DevKit V1")
 		(property "Reference" "A1"
-			(at 12.7 -8.5 0)
+			(at 12.7 -10.5 0)
 			(layer "F.SilkS")
 			(effects
@@
 		(tags "terminal block bornier3")
 		(property "Reference" "J8"
-			(at 5.05 -4.65 0)
+			(at 5.05 -6.65 0)
 			(layer "F.SilkS")
 			(effects
@@
 		(tags "Through hole pin header THT 1x06 2.54mm single row")
 		(property "Reference" "J19"
-			(at 0 -2.33 0)
+			(at 0 -4.33 0)
 			(layer "F.SilkS")
 			(effects
@@
 		(tags "Through hole socket strip THT 1x04 2.54mm single row")
 		(property "Reference" "J14"
-			(at 0 -2.77 0)
+			(at 0 -4.27 0)
 			(layer "F.SilkS")
 			(effects
@@
 		(tags "terminal block bornier3")
 		(property "Reference" "J4"
-			(at 5.05 -4.65 0)
+			(at 5.05 -6.65 0)
 			(layer "F.SilkS")
 			(effects
@@
 		(tags "terminal block bornier3")
 		(property "Reference" "J3"
-			(at 5.05 -4.65 0)
+			(at 5.05 -6.65 0)
 			(layer "F.SilkS")
 			(effects
@@
 		(tags "terminal block bornier3")
 		(property "Reference" "J12"
-			(at 5.05 -4.65 0)
+			(at 5.05 -6.65 0)
 			(layer "F.SilkS")
 			(effects
@@
 		(tags "Through hole socket strip THT 1x04 2.54mm single row")
 		(property "Reference" "J16"
-			(at 0 -2.77 0)
+			(at 0 -4.27 0)
 			(layer "F.SilkS")
 			(effects
@@
 		(tags "connector JST XH vertical")
 		(property "Reference" "J13"
-			(at 2.5 -3.55 0)
+			(at 2.5 -2.55 0)
 			(layer "F.SilkS")
 			(effects
@@
 		(layer "Edge.Cuts")
 	)
+	(gr_text "JLCJLCJLCJLC"
+		(at 64 145.5 0)
+		(layer "B.SilkS")
+		(effects
+			(font
+				(size 1 1)
+				(thickness 0.16)
+			)
+			(justify mirror)
+		)
+	)
 	(gr_text "ANTENNE WIFI : zone degagee (pas de cuivre dessous)"
 		(at 90.7 98.5 0)
@@
 		(effects
 			(font
-				(size 0.8 0.8)
-				(thickness 0.12)
+				(size 1 1)
+				(thickness 0.16)
 			)
 		)
@@
 		(effects
 			(font
-				(size 0.8 0.8)
-				(thickness 0.12)
+				(size 1 1)
+				(thickness 0.16)
 			)
 		)
@@
 			(font
 				(size 1 1)
-				(thickness 0.15)
+				(thickness 0.16)
 			)
 		)
@@
 		(effects
 			(font
-				(size 0.8 0.8)
-				(thickness 0.12)
+				(size 1 1)
+				(thickness 0.16)
 			)
 		)
@@
 		(effects
 			(font
-				(size 0.8 0.8)
-				(thickness 0.12)
+				(size 1 1)
+				(thickness 0.16)
 			)
 		)
@@
 			(font
 				(size 1 1)
-				(thickness 0.15)
+				(thickness 0.16)
 			)
 		)
@@
 		(effects
 			(font
-				(size 0.8 0.8)
-				(thickness 0.12)
+				(size 1 1)
+				(thickness 0.16)
 			)
 		)
@@
 		(effects
 			(font
-				(size 0.8 0.8)
-				(thickness 0.12)
+				(size 1 1)
+				(thickness 0.16)
 			)
 		)
@@
 		(effects
 			(font
-				(size 0.8 0.8)
-				(thickness 0.12)
+				(size 1 1)
+				(thickness 0.16)
 			)
 		)
@@
 		(effects
 			(font
-				(size 0.8 0.8)
-				(thickness 0.12)
+				(size 1 1)
+				(thickness 0.16)
 			)
 		)
@@
 		(effects
 			(font
-				(size 0.8 0.8)
-				(thickness 0.12)
+				(size 1 1)
+				(thickness 0.16)
 			)
 		)
@@
 		(effects
 			(font
-				(size 0.8 0.8)
-				(thickness 0.12)
+				(size 1 1)
+				(thickness 0.16)
 			)
 		)
@@
 		(effects
 			(font
-				(size 0.8 0.8)
-				(thickness 0.12)
+				(size 1 1)
+				(thickness 0.16)
 			)
 		)
@@
 		(effects
 			(font
-				(size 0.8 0.8)
-				(thickness 0.12)
+				(size 1 1)
+				(thickness 0.16)
 			)
 		)
@@
 		(effects
 			(font
-				(size 0.8 0.8)
-				(thickness 0.12)
+				(size 1 1)
+				(thickness 0.16)
 			)
 		)
@@
 			(font
 				(size 1.2 1.2)
-				(thickness 0.18)
+				(thickness 0.19)
 			)
 		)
@@
 		(effects
 			(font
-				(size 0.8 0.8)
-				(thickness 0.12)
+				(size 1 1)
+				(thickness 0.16)
 			)
 		)
@@
 		(effects
 			(font
-				(size 0.8 0.8)
-				(thickness 0.12)
+				(size 1 1)
+				(thickness 0.16)
 			)
 		)
@@
 		(effects
 			(font
-				(size 0.8 0.8)
-				(thickness 0.12)
+				(size 1 1)
+				(thickness 0.16)
 			)
 		)
@@
 			(font
 				(size 1 1)
-				(thickness 0.15)
+				(thickness 0.16)
 			)
 		)
@@
 		(effects
 			(font
-				(size 0.8 0.8)
-				(thickness 0.12)
+				(size 1 1)
+				(thickness 0.16)
 			)
 		)
@@
 		(effects
 			(font
-				(size 0.8 0.8)
-				(thickness 0.12)
+				(size 1 1)
+				(thickness 0.16)
 			)
 		)
@@
 		(effects
 			(font
-				(size 0.8 0.8)
-				(thickness 0.12)
+				(size 1 1)
+				(thickness 0.16)
 			)
 		)
@@
 		(effects
 			(font
-				(size 0.8 0.8)
-				(thickness 0.12)
+				(size 1 1)
+				(thickness 0.16)
 			)
 		)
@@
 			(font
 				(size 1 1)
-				(thickness 0.15)
+				(thickness 0.16)
 			)
 		)
@@
 		(effects
 			(font
-				(size 0.8 0.8)
-				(thickness 0.12)
+				(size 1 1)
+				(thickness 0.16)
 			)
 		)
@@
 		(effects
 			(font
-				(size 0.8 0.8)
-				(thickness 0.12)
+				(size 1 1)
+				(thickness 0.16)
 			)
 		)
@@
 		(effects
 			(font
-				(size 0.8 0.8)
-				(thickness 0.12)
+				(size 1 1)
+				(thickness 0.16)
 			)
 		)
@@
 		(effects
 			(font
-				(size 0.8 0.8)
-				(thickness 0.12)
+				(size 1 1)
+				(thickness 0.16)
 			)
 		)
@@
 			(font
 				(size 1 1)
-				(thickness 0.15)
+				(thickness 0.16)
 			)
 		)
@@
 		(effects
 			(font
-				(size 0.8 0.8)
-				(thickness 0.12)
+				(size 1 1)
+				(thickness 0.16)
 			)
 		)
@@
 			(font
 				(size 1 1)
-				(thickness 0.15)
+				(thickness 0.16)
 			)
 		)
@@
 		(effects
 			(font
-				(size 0.8 0.8)
-				(thickness 0.12)
+				(size 1 1)
+				(thickness 0.16)
 			)
 		)
@@
 			(font
 				(size 1.5 1.5)
-				(thickness 0.22)
+				(thickness 0.24)
 			)
 		)

Commit message: feat(hardware): carte commune rev 0.2 — rail capteurs commuté par GPIO13, veille à ~0
L'audit des sources n3pp/msp a montré que GPIO13 (RELAIS) n'est PAS une sortie
relais métier : c'est un POWER-GATE — mis à 1 en tout début de setup(), réaffirmé
à chaque réveil (callback connectWifi des deux séquenceurs), jamais écrit à 0,
non piloté par le serveur, relâché en deep sleep. La rev 0.1 le câblait sur un
relais générique et laissait capteurs/OLED/pull-ups sur le 3V3 permanent :
régression vs les montages actuels. La rev 0.2 restitue l'architecture réelle :

- rail scindé +3V3 (DevKit) / +3V3_SW (TOUT le reste : borniers ADC, 3 DHT,
  DS18B20, pluie, OLED, 3 ports I2C, rail Dupont J19 — ET leurs pull-ups,
  sinon phantom power par les lignes de données)
- interrupteur HAUT P-MOSFET : Q7 NDP6020P piloté par l'étage GPIO13 existant
  (R1 1k + R5 10k + Q1 BC337) + R36 100k (rail coupé par défaut) — zéro
  bobine (le relais SRD consommait 72 mA tout l'éveil), zéro usure
- pont diviseur batterie commuté côté HAUT (Q8 BS250 + Q9 BC337 + R37/R38
  100k) : ~0,85 mA économisés en veille, et jamais plus de 3,3 V sur GPIO36
  pont coupé (une coupure basse aurait laissé VBAT remonter par R34)
- C5 470 µF réservoir sur +3V3 (pointes WiFi en alim batterie/LDO 250 mA)
- JP1 : cavalier isolant J29 (entrée LDO batterie) du rail 3V3 pour flasher
  en USB sans mettre deux régulateurs en parallèle
- la carte passe de 6 à 5 canaux relais (REL2 pompe n3pp + 4 AUX) — le
  6e « relais » n'a jamais existé côté firmware

Firmwares INCHANGÉS (GPIO13 garde sa sémantique). Checker anti-dérive étendu :
topologie power-gate + pont commuté vérifiées contre les sources. Amorces de
routage SEED_TRACKS intégrées à route_lv.py (AUX6 pincé sous la zone antenne,
échec freerouting reproductible sans elles).

Validation : ERC 0 erreur, DRC 0 violation / 0 pad non connecté, checker OK
(21 signaux), sérigraphie 0 conflit, gerbers v0.2 (10 fichiers, 404+4 perçages).
Docs à jour : README, ACHATS (BOM socle rev 0.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
Parts:
- removed D1: 1N4007, n3commun:D_DO-41_SOD81_P10.16mm_Horizontal
- removed J3: Bornier_5.08, n3commun:TerminalBlock_bornier-3_P5.08mm
- removed K1: SRD-05VDC-SL-C, n3commun:Relay_SPDT_SANYOU_SRD_Series_Form_C
- added C5: 470u/16V, n3commun:CP_Radial_D8.0mm_P3.50mm, F.Cu at (68.0, 141.0)
- added JP1: Jumper, n3commun:PinHeader_1x02_P2.54mm_Vertical, F.Cu at (227.0, 131.0)
- added Q7: NDP6020P, n3commun:TO-220-3_Vertical, F.Cu at (58.0, 55.0)
- added Q8: BS250, n3commun:TO-92_Inline, F.Cu at (52.0, 68.0)
- added Q9: BC337-40, n3commun:TO-92_Inline, F.Cu at (62.0, 68.0)
- added R36: 100k, n3commun:R_Axial_DIN0207_L6.3mm_D2.5mm_P10.16mm_Horizontal, F.Cu at (54.0, 62.0)
- added R37: 100k, n3commun:R_Axial_DIN0207_L6.3mm_D2.5mm_P10.16mm_Horizontal, F.Cu at (52.0, 74.0)
- added R38: 100k, n3commun:R_Axial_DIN0207_L6.3mm_D2.5mm_P10.16mm_Horizontal, F.Cu at (52.0, 80.0)
Connections:
- net REL1_B renamed PWR_B
- net REL1_LED renamed RAIL_LED
- C3 pad 1: +3V3 -> +3V3_SW
- C4 pad 1: +3V3 -> +3V3_SW
- J10 pad 1: +3V3 -> +3V3_SW
- J11 pad 1: +3V3 -> +3V3_SW
- J12 pad 1: +3V3 -> +3V3_SW
- J13 pad 1: +3V3 -> +3V3_SW
- J14 pad 2: +3V3 -> +3V3_SW
- J15 pad 2: +3V3 -> +3V3_SW
- J16 pad 2: +3V3 -> +3V3_SW
- J17 pad 2: +3V3 -> +3V3_SW
- J19 pad 5: +3V3 -> +3V3_SW
- J19 pad 6: +3V3 -> +3V3_SW
- J22 pad 1: +3V3 -> +3V3_SW
- J23 pad 1: +3V3 -> +3V3_SW
- J24 pad 1: +3V3 -> +3V3_SW
- J25 pad 1: +3V3 -> +3V3_SW
- J26 pad 1: +3V3 -> +3V3_SW
- J29 pad 1: +3V3 -> +3V3_IN
- J9 pad 1: +3V3 -> +3V3_SW
- LED1 pad 1: REL1_SW -> GND
- Q1 pad 1: REL1_SW -> PWR_G
- R21 pad 1: +3V3 -> +3V3_SW
- R22 pad 1: +3V3 -> +3V3_SW
- R23 pad 1: +3V3 -> +3V3_SW
- R24 pad 1: +3V3 -> +3V3_SW
- R25 pad 1: +3V3 -> +3V3_SW
- R26 pad 1: +3V3 -> +3V3_SW
- R34 pad 1: VBAT -> VBAT_SW
- R9 pad 1: +5V -> +3V3_SW
Routing:
- net GND: track 1392.4 -> 692.0 mm, vias 85 -> 91
- net +3V3_SW: track 0.00 -> 497.3 mm, vias 0 -> 2
- net VBAT_SW: track 0.00 -> 185.5 mm, vias 0 -> 1
- net VBAT: track 9.66 -> 189.3 mm, vias 0 -> 1
- net +3V3: track 336.7 -> 287.9 mm, vias 0 -> 1
- net +5V: track 642.0 -> 593.3 mm
- net PWR_G: track 0.00 -> 46.1 mm, vias 0 -> 1
- net REL1_NO: track 40.9 -> 0.00 mm
- net SERVOGD_GPIO25: track 176.5 -> 214.5 mm
- net REL1_SW: track 35.3 -> 0.00 mm
- net ADC_C_GPIO35: track 113.3 -> 85.6 mm
- net DHT_EXT_GPIO15: track 71.4 -> 51.2 mm, vias 0 -> 1
- net REL3_B: track 22.9 -> 40.8 mm
- net REL4_B: track 22.9 -> 40.8 mm
- net REL1_COM: track 16.9 -> 0.00 mm
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Other:
- board text added: "CARTE COMMUNE n3pp + msp v0.2"
- board text added: "JP1 3V3"
- board text added: "PWR CAPTEURS GPIO13"
- board text removed: "CARTE COMMUNE n3pp + msp v0.1"
- board text removed: "REL1 GPIO13 COMMUN"
