File: hardware/n3pp-msp-commun/kicad/n3pp-msp-commun.kicad_sch (KiCad schematic)
At the start: 94 parts, among them J1 Bornier_5.08, J10 JST-XH, J11 JST-XH, J12 Bornier_5.08, J13 JST-XH, J14 Support OLED, J15 Support I2C libre, J16 Support I2C libre, J17 Support I2C libre, J18 Header GPIO libres, J19 Rail alim Dupont, J2 Jack 5.5/2.1, J20 Header servo, J21 Header servo, J22 Bornier_5.08, J23 Bornier_5.08, J24 Bornier_5.08, J25 Bornier_5.08, J26 Bornier_5.08, J27 Bornier_5.08, J28 Bornier_5.08, J29 Bornier_5.08, J3 Bornier_5.08, J4 Bornier_5.08, J5 Bornier_5.08, J6 Bornier_5.08, J7 Bornier_5.08, J8 Bornier_5.08, J9 JST-XH, K1 SRD-05VDC-SL-C, K2 SRD-05VDC-SL-C, K3 SRD-05VDC-SL-C, K4 SRD-05VDC-SL-C, K5 SRD-05VDC-SL-C, K6 SRD-05VDC-SL-C, Q1 BC337-40, Q2 BC337-40, Q3 BC337-40, Q4 BC337-40, Q5 BC337-40, Q6 BC337-40

Commit message: feat(hardware): carte commune rev 0.2 — rail capteurs commuté par GPIO13, veille à ~0
L'audit des sources n3pp/msp a montré que GPIO13 (RELAIS) n'est PAS une sortie
relais métier : c'est un POWER-GATE — mis à 1 en tout début de setup(), réaffirmé
à chaque réveil (callback connectWifi des deux séquenceurs), jamais écrit à 0,
non piloté par le serveur, relâché en deep sleep. La rev 0.1 le câblait sur un
relais générique et laissait capteurs/OLED/pull-ups sur le 3V3 permanent :
régression vs les montages actuels. La rev 0.2 restitue l'architecture réelle :

- rail scindé +3V3 (DevKit) / +3V3_SW (TOUT le reste : borniers ADC, 3 DHT,
  DS18B20, pluie, OLED, 3 ports I2C, rail Dupont J19 — ET leurs pull-ups,
  sinon phantom power par les lignes de données)
- interrupteur HAUT P-MOSFET : Q7 NDP6020P piloté par l'étage GPIO13 existant
  (R1 1k + R5 10k + Q1 BC337) + R36 100k (rail coupé par défaut) — zéro
  bobine (le relais SRD consommait 72 mA tout l'éveil), zéro usure
- pont diviseur batterie commuté côté HAUT (Q8 BS250 + Q9 BC337 + R37/R38
  100k) : ~0,85 mA économisés en veille, et jamais plus de 3,3 V sur GPIO36
  pont coupé (une coupure basse aurait laissé VBAT remonter par R34)
- C5 470 µF réservoir sur +3V3 (pointes WiFi en alim batterie/LDO 250 mA)
- JP1 : cavalier isolant J29 (entrée LDO batterie) du rail 3V3 pour flasher
  en USB sans mettre deux régulateurs en parallèle
- la carte passe de 6 à 5 canaux relais (REL2 pompe n3pp + 4 AUX) — le
  6e « relais » n'a jamais existé côté firmware

Firmwares INCHANGÉS (GPIO13 garde sa sémantique). Checker anti-dérive étendu :
topologie power-gate + pont commuté vérifiées contre les sources. Amorces de
routage SEED_TRACKS intégrées à route_lv.py (AUX6 pincé sous la zone antenne,
échec freerouting reproductible sans elles).

Validation : ERC 0 erreur, DRC 0 violation / 0 pad non connecté, checker OK
(21 signaux), sérigraphie 0 conflit, gerbers v0.2 (10 fichiers, 404+4 perçages).
Docs à jour : README, ACHATS (BOM socle rev 0.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
Parts:
- removed D1: 1N4007, n3commun:D_DO-41_SOD81_P10.16mm_Horizontal, symbol n3commun:D
- removed J3: Bornier_5.08, n3commun:TerminalBlock_bornier-3_P5.08mm, symbol n3commun:CONN_03
- removed K1: SRD-05VDC-SL-C, n3commun:Relay_SPDT_SANYOU_SRD_Series_Form_C, symbol n3commun:RELAY_SRD
- added C5: 470u/16V, n3commun:CP_Radial_D8.0mm_P3.50mm, symbol n3commun:CP
- added JP1: Jumper, n3commun:PinHeader_1x02_P2.54mm_Vertical, symbol n3commun:CONN_02
- added Q7: NDP6020P, n3commun:TO-220-3_Vertical, symbol n3commun:PMOS_GDS
- added Q8: BS250, n3commun:TO-92_Inline, symbol n3commun:PMOS_DGS
- added Q9: BC337-40, n3commun:TO-92_Inline, symbol n3commun:NPN
- added R36, R37, R38: 100k, n3commun:R_Axial_DIN0207_L6.3mm_D2.5mm_P10.16mm_Horizontal, symbol n3commun:R
Connections:
- net +3V3: now also C5.1 (+), JP1.2, Q7.3 (S), R36.1; no longer C3.1, C4.1, J10.1, J11.1, J12.1, J13.1, J14.2, J15.2, J16.2, J17.2, J19.5, J19.6, J22.1, J23.1, J24.1, J25.1, J26.1, J29.1, J9.1, R21.1, R22.1, R23.1, R24.1, R25.1, R26.1
- net +5V: no longer R9.1
- net GND: now also LED1.1 (K), C5.2 (-), Q9.3 (E)
- net VBAT: now also Q8.3 (S), R37.1; no longer R34.1
- net REL1_B renamed PWR_B
- net REL1_LED renamed RAIL_LED
- net REL1_SW renamed PWR_G
- net PWR_G: now also Q7.1 (G), R36.2; no longer LED1.1 (K)
- new net +3V3_IN: J29.1, JP1.1
- new net +3V3_SW: C3.1, C4.1, J10.1, J11.1, J12.1, J13.1, J14.2, J15.2, J16.2, J17.2, J19.5, J19.6, J22.1, J23.1, J24.1, J25.1, J26.1, J9.1, Q7.2 (D), R21.1, R22.1, R23.1, R24.1, R25.1, R26.1, R38.1, R9.1
- new net PDIV_B: Q9.2 (B), R38.2
- new net PDIV_G: Q8.2 (G), Q9.1 (C), R37.2
- new net VBAT_SW: Q8.1 (D), R34.1
Other:
- note added: "5 ENTREES ANALOGIQUES ADC1 (compatibles WiFi) — bornier 3V3_SW/AIN/GND. 10k bas de pont : peupler pour une LDR, DNP pour un capteur à sortie AO. A=33 B=32 C=35 D=34 E=39 (35/34/39 = entrées seules)."
- note added: "BATTERIE : pont 2.2k/2.2k -> GPIO36 (VP), COMMUTE par Q8/Q9 (actif seulement rail capteurs allumé : ~0 conso en veille). J27 = VBAT/GND (valeurs n3_defaults.h : N3_BATTERY_R1/R2)."
- note added: "DISTRIBUTION : rail J19 (2x5V 2xGND 2x3V3_SW, coupé en veille) + borniers J28 (5V) et J29 (3V3). J29 = AUSSI l'entrée LDO batterie, via JP1 — retirer le cavalier pour flasher en USB sur station batterie."
- note added: "INTERRUPTEUR D'ALIM CAPTEURS + 5 RELAIS 5V (actifs HAUT). GPIO13 (RELAIS, les 2 firmwares) = power-gate : 1 au réveil, relâché en deep sleep -> Q1+Q7 (P-MOSFET) coupent le rail +3V3_SW (capteurs, OLED, I2C, pull-ups) pendant la veille. REL2 GPIO12 = POMPE (n3pp, strapping MTDI -> pull-down 10k) ; REL3..REL6 = AUX GPIO16/17/19/23 (extension)."
- note removed: "5 ENTREES ANALOGIQUES ADC1 (compatibles WiFi) — bornier 3V3/AIN/GND. 10k bas de pont : peupler pour une LDR, DNP pour un capteur à sortie AO. A=33 B=32 C=35 D=34 E=39 (35/34/39 = entrées seules)."
- note removed: "6 RELAIS 5V — commande ACTIVE HAUT. REL1 GPIO13 = RELAIS (n3pp ET msp) ; REL2 GPIO12 = POMPE (n3pp, strapping MTDI -> pull-down base 10k = état sûr au boot) ; REL3..REL6 = AUX GPIO16/17/19/23 (extension, non pilotés par les firmwares actuels — pattern AUX1/AUX2 de ffp5cs)."
- note removed: "BATTERIE : pont 2.2k/2.2k -> GPIO36 (VP, entrée seule). J27 = VBAT/GND (valeurs n3_defaults.h : N3_BATTERY_R1/R2)."
- note removed: "DISTRIBUTION : rail J19 (2x5V 2xGND 2x3V3) + borniers J28 (5V) et J29 (3V3)."
- moved on the sheet: R9
