File: hardware/n3-universal/kicad/n3-universal.kicad_pcb (KiCad board)
At the start: 2 copper layers, 278 x 120 mm, 131 parts, among them J1 Bornier_5.08, J10 JST-XH, J11 Bornier_5.08, J12 Bornier_5.08, J13 Support OLED, J14 Support I2C ext, J15 Header servo, J16 Header servo, J17 Header service, J18 Bornier_5.08, J19 Bornier_5.08, J2 Jack 5.5/2.1, J20 Header alim, J21 Support I2C libre, J22 Support I2C libre, J23 Bornier_5.08, J24 Bornier_5.08, J25 Bornier_5.08, J26 Bornier_5.08, J27 Bornier_5.08, J28 Support I2C libre, J29 JST-XH, J3 Bornier_5.08, J30 JST-XH, J31 Bornier_5.08, J32 Bornier_5.08, J33 Bornier_5.08, J34 Bornier_5.08, J35 Support module microSD, J36 Bornier_5.08, J37 Bornier_5.08, J4 Bornier_5.08, J5 Bornier_5.08, J6 Bornier_5.08, J7 JST-XH, J8 JST-XH, J9 JST-XH, K1 SRD-05VDC-SL-C, K2 SRD-05VDC-SL-C, K3 SRD-05VDC-SL-C, K4 SRD-05VDC-SL-C, K5 SRD-05VDC-SL-C, K6 SRD-05VDC-SL-C, Q1 BC337-40, Q10 BC337-40, Q11 NDP6020P, Q2 BC337-40, Q3 BC337-40, Q4 BC337-40, Q5 BC337-40, Q6 BC337-40, Q7 NDP6020P, Q8 BC337-40, Q9 BS250

Commit message: fix(n3-universal): corrections de l'audit final — Q11, coin PSU 230V, plan GND, H1, poses conditionnelles + contrats serveur (n3pp 4.72, ffp5cs 15.29)
Audit exhaustif multi-axes (netlist alim/signaux, strapping, géométrie secteur,
firmwares, contrats serveur) avant commande. Corrections carte (PCB routé,
schéma régénéré, générateur synchronisé, gerbers/PDF/SVG re-exportés — PTH 521) :

- Q11 (anti-inversion bus 12V) : câblé au brochage BS250 (D-G-S), l'entrée 12 V
  arrivait sur la GRILLE du NDP6020P (TO-220 : 1=G 2=D 3=S) — profil 12 V
  inopérant et Vgs hors spec. Recâblé G/D/S comme Q7 ; liaisons re-routées B.Cu.
- Coin PSU 230 V re-routé : L passait à 0,75 mm du pad neutre de J27 (tronçon
  non fusé), N // LF à 1,5 mm. Nouveau tracé avec écarts L<->N<->LF >= 3 mm hors
  pas des composants ; J27 devient 1=N / 2=L, repères L/N sérigraphiés.
- Plan GND exclu du coin PSU (246..318 x 40..73, F+B) : il coulait sous les
  pistes/pads 230 V ; check_mains_gap voit désormais les ZONES REMPLIES
  (il était aveugle au cuivre coulé) — 0 violation.
- H1 (coin relais, enclavé par K1) : vis NYLON obligatoire (tête métal à
  ~4,3 mm du 230 V) — keepout de coulée sous la tête + sérigraphie H1=NYLON.
- Poses conditionnelles (BOM étoilée) : R17/R18/R19 (2k, ponts écho HC-SR04)
  posées ffp5cs uniquement — permanentes, elles verrouillaient PLUIE/US1 à
  « mouillé » et rendaient DHT_EXT/US2 illisible côté msp (niveau haut ~0,55 V) ;
  R27 (10k) posée pour LDR seulement (module AO msp atténué de moitié sinon).
- microSD/MTDI : module 3,3 V direct sans tampon, réservé S3 ; sur WROOM efuse
  VDD_SDIO=3V3 obligatoire (une carte SD peut tirer GPIO12 haut au boot).
  Étiquettes servo égarées en zone secteur repositionnées ; JP1 « 1-2 » précisé.

Contrats serveur (croisements découverts par l'audit) :
- n3pp v4.72 : clé JSON pompe découplée de la broche (POMPE_OUTPUT_KEY="12" —
  en universel POMPE=16 lisait une ligne legacy non exposée par l'UI).
- ffp5cs v15.29 : gpio_mapping.h reprend le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
Parts:
- R17, R18, R19: value 2k -> 2k*
- R27: value 10k -> 10k*
Connections:
- J27 pad 1: MAINS_L -> MAINS_N
- J27 pad 2: MAINS_N -> MAINS_L
- Q11 pad 1: VBAT12_IN -> QP_G
- Q11 pad 2: QP_G -> VBAT12_IN
Routing:
- net VBAT12_IN: track 20.3 -> 35.5 mm, vias 0 -> 1
- net MAINS_L: track 21.0 -> 11.1 mm
- net MAINS_N: track 57.5 -> 64.1 mm
- net MAINS_LF: track 66.4 -> 67.5 mm
- net QP_G: track 19.4 -> 18.8 mm
Other:
- board text added: "H1=NYLON"
- board text added: "JP1 BYPASS 1-2: FERME=rail permanent (ffp5cs)"
- board text added: "L"
- board text added: "N"
- board text removed: "JP1 BYPASS: FERME=rail permanent (ffp5cs)"
Changed lines of the file:
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@@
 			)
 		)
-		(property "Value" "2k"
+		(property "Value" "2k*"
 			(at 5.08 2.37 0)
 			(layer "F.Fab")
@@
 			)
 		)
-		(property "Value" "2k"
+		(property "Value" "2k*"
 			(at 5.08 2.37 0)
 			(layer "F.Fab")
@@
 			)
 			(remove_unused_layers no)
-			(net 87 "VBAT12_IN")
+			(net 31 "QP_G")
 		)
 		(pad "2" thru_hole oval
@@
 			)
 			(remove_unused_layers no)
-			(net 31 "QP_G")
+			(net 87 "VBAT12_IN")
 		)
 		(pad "3" thru_hole oval
@@
 			)
 			(remove_unused_layers no)
-			(net 24 "MAINS_L")
+			(net 26 "MAINS_N")
 		)
 		(pad "2" thru_hole circle
@@
 			)
 			(remove_unused_layers no)
-			(net 26 "MAINS_N")
+			(net 24 "MAINS_L")
 		)
 		(model "${KICAD8_3DMODEL_DIR}/TerminalBlock.3dshapes/TerminalBlock_bornier-2_P5.08mm.wrl"
@@
 			)
 		)
-		(property "Value" "10k"
+		(property "Value" "10k*"
 			(at 5.08 2.37 0)
 			(layer "F.Fab")
@@
 		(tags "to-92 sc-43 sc-43a sot54 PA33 transistor")
 		(property "Reference" "Q9"
-			(at 1.27 -3.56 0)
+			(at 1.27 -4.06 0)
 			(layer "F.SilkS")
 			(effects
@@
 			)
 		)
-		(property "Value" "2k"
+		(property "Value" "2k*"
 			(at 5.08 2.37 0)
 			(layer "F.Fab")
@@
 	)
 	(gr_text "SRV GROS"
-		(at 266 55 0)
+		(at 297 105.5 0)
 		(layer "F.SilkS")
 		(effects
@@
 	)
 	(gr_text "SRV PETITS"
-		(at 266 67 0)
+		(at 297 127.5 0)
 		(layer "F.SilkS")
 		(effects
@@
 		)
 	)
-	(gr_text "JP1 BYPASS: FERME=rail permanent (ffp5cs)"
+	(gr_text "JP1 BYPASS 1-2: FERME=rail permanent (ffp5cs)"
 		(at 238 111 0)
 		(layer "F.SilkS")
@@
 		)
 	)
+	(gr_text "H1=NYLON"
+		(at 44.3 55 0)
+		(layer "F.SilkS")
+		(effects
+			(font
+				(size 1 1)
+				(thickness 0.15)
+			)
+		)
+	)
 	(gr_text "NC COM NO"
 		(at 160 57.5 0)
@@
 		)
 	)
+	(gr_text "N"
+		(at 250 41.6 0)
+		(layer "F.SilkS")
+		(effects
+			(font
+				(size 1 1)
+				(thickness 0.15)
+			)
+		)
+	)
 	(gr_text "SD"
 		(at 209 139.5 0)
@@
 		)
 	)
+	(gr_text "L"
+		(at 256.8 41.6 0)
+		(layer "F.SilkS")
+		(effects
+			(font
+				(size 1 1)
+				(thickness 0.15)
+			)
+		)
+	)
 	(gr_text "K1 POMPE AQUA/ARROSAGE"
 		(at 58 43 0)
@@
 	)
 	(segment
-		(start 266 42.5)
+		(start 255.08 46)
 		(end 266 44)
 		(width 2.5)
@@
 	)
 	(segment
-		(start 250 46)
-		(end 250 42.5)
-		(width 2.5)
-		(layer "F.Cu")
-		(net 24)
-	)
-	(segment
-		(start 250 42.5)
-		(end 266 42.5)
-		(width 2.5)
-		(layer "F.Cu")
-		(net 24)
-	)
-	(segment
 		(start 266 66.5)
-		(end 260 66.5)
-		(width 2.5)
-		(layer "F.Cu")
-		(net 25)
-	)
-	(segment
-		(start 299 54)
-		(end 303 50)
+		(end 303 66.5)
 		(width 2.5)
 		(layer "F.Cu")
@@
 	)
 	(segment
-		(start 270 54)
-		(end 299 54)
-		(width 2.5)
-		(layer "F.Cu")
-		(net 25)
-	)
-	(segment
-		(start 270 66.5)
-		(end 270 54)
-		(width 2.5)
-		(layer "F.Cu")
-		(net 25)
-	)
-	(segment
-		(start 260 66.5)
-		(end 258 64)
-		(width 2.5)
-		(layer "F.Cu")
-		(net 25)
-	)
-	(segment
-		(start 303 50)
+		(start 303 66.5)
 		(end 303 46)
 		(width 2.5)
@@
 	)
 	(segment
-		(start 266 66.5)
-		(end 270 66.5)
-		(width 2.5)
-		(layer "F.Cu")
-		(net 25)
-	)
-	(segment
-		(start 258 64)
+		(start 262 66.5)
 		(end 258 62)
 		(width 2.5)
@@
 	)
 	(segment
-		(start 290 50)
-		(end 294 46)
+		(start 266 66.5)
+		(end 262 66.5)
 		(width 2.5)
 		(layer "F.Cu")
-		(net 26)
+		(net 25)
 	)
 	(segment
-		(start 255.08 50)
-		(end 290 50)
+		(start 250 46)
+		(end 250 60)
 		(width 2.5)
 		(layer "F.Cu")
@@
 	)
 	(segment
-		(start 255.08 58)
-		(end 253 60)
+		(start 250 52)
+		(end 288 52)
 		(width 2.5)
 		(layer "F.Cu")
@@
 	)
 	(segment
-		(start 255.08 46)
-		(end 255.08 58)
+		(start 250 60)
+		(end 253 62)
 		(width 2.5)
 		(layer "F.Cu")
@@
 	)
 	(segment
-		(start 253 60)
-		(end 253 62)
+		(start 288 52)
+		(end 294 46)
 		(width 2.5)
 		(layer "F.Cu")
@@
 	)
 	(segment
-		(start 232.5983 144.0583)
-		(end 232.5983 129.4017)
+		(start 234 128)
+		(end 232 130)
 		(width 0.4)
 		(layer "B.Cu")
@@
 	)
 	(segment
-		(start 234.54 146)
-		(end 232.5983 144.0583)
-		(width 0.4)
-		(layer "B.Cu")
-		(net 31)
-	)
-	(segment
-		(start 232.5983 129.4017)
-		(end 234 128)
+		(start 232 130)
+		(end 232 146)
 		(width 0.4)
 		(layer "B.Cu")
@@
 	)
 	(segment
-		(start 220.108 153.3098)
-		(end 222.936 153.3098)
+		(start 216 151)
+		(end 216 157)
 		(width 1.2)
-		(layer "B.Cu")
+		(layer "F.Cu")
 		(net 87)
 	)
 	(segment
-		(start 218.3017 151)
-		(end 218.3017 151.5035)
+		(start 227 157)
+		(end 227 152.8)
 		(width 1.2)
-		(layer "B.Cu")
+		(layer "F.Cu")
 		(net 87)
 	)
 	(segment
-		(start 218.3017 151.5035)
-		(end 220.108 153.3098)
+		(start 216 157)
+		(end 227 157)
 		(width 1.2)
-		(layer "B.Cu")
+		(layer "F.Cu")
+		(net 87)
+	)
+	(via
+		(at 227 152.8)
+		(size 0.8)
+		(drill 0.4)
+		(layers "F.Cu" "B.Cu")
 		(net 87)
 	)
 	(segment
-		(start 222.936 153.3098)
-		(end 230.2458 146)
+		(start 234.54 148)
+		(end 234.54 146)
 		(width 1.2)
 		(layer "B.Cu")
@@
 	)
 	(segment
-		(start 216 151)
-		(end 218.3017 151)
+		(start 227 148)
+		(end 234.54 148)
 		(width 1.2)
 		(layer "B.Cu")
@@
 	)
 	(segment
-		(start 232 146)
-		(end 230.2458 146)
+		(start 227 152.8)
+		(end 227 148)
 		(width 1.2)
 		(layer "B.Cu")
@@
 		(polygon
 			(pts
-				(xy 40 40) (xy 45.2 40) (xy 45.2 84) (xy 246 84) (xy 246 40) (xy 318 40) (xy 318 160) (xy 40 160)
+				(xy 40 40) (xy 45.2 40) (xy 45.2 84) (xy 246 84) (xy 246 73) (xy 318 73) (xy 318 160) (xy 40 160)
 			)
 		)
@@
 	)
 	(zone
+		(net 0)
+		(net_name "")
+		(layers "F.Cu" "B.Cu")
+		(hatch edge 0.5)
+		(connect_pads
+			(clearance 0)
+		)
+		(min_thickness 0.25)
+		(filled_areas_thickness no)
+		(keepout
+			(tracks allowed)
+			(vias allowed)
+			(pads allowed)
+			(copperpour not_allowed)
+			(footprints allowed)
+		)
+		(fill
+			(thermal_gap 0.5)
+			(thermal_bridge_width 0.5)
+		)
+		(polygon
+			(pts
+				(xy 41 41) (xy 49 41) (xy 49 49) (xy 41 49)
+			)
+		)
+	)
+	(zone
 		(net 15)
 		(net_name "GND")
@@
 		(polygon
 			(pts
-				(xy 40 40) (xy 45.2 40) (xy 45.2 84) (xy 246 84) (xy 246 40) (xy 318 40) (xy 318 160) (xy 40 160)
+				(xy 40 40) (xy 45.2 40) (xy 45.2 84) (xy 246 84) (xy 246 73) (xy 318 73) (xy 318 160) (xy 40 160)
 			)
 		)
