File: hardware/n3-universal/kicad/n3-universal.kicad_pcb (KiCad board)
At the start: 2 copper layers, 278 x 120 mm, 131 parts, among them J1 Bornier_5.08, J10 JST-XH, J11 Bornier_5.08, J12 Bornier_5.08, J13 Support OLED, J14 Support I2C ext, J15 Header servo, J16 Header servo, J17 Header service, J18 Bornier_5.08, J19 Bornier_5.08, J2 Jack 5.5/2.1, J20 Header alim, J21 Support I2C libre, J22 Support I2C libre, J23 Bornier_5.08, J24 Bornier_5.08, J25 Bornier_5.08, J26 Bornier_5.08, J27 Bornier_5.08, J28 Support I2C libre, J29 JST-XH, J3 Bornier_5.08, J30 JST-XH, J31 Bornier_5.08, J32 Bornier_5.08, J33 Bornier_5.08, J34 Bornier_5.08, J35 Support module microSD, J36 Bornier_5.08, J37 Bornier_5.08, J4 Bornier_5.08, J5 Bornier_5.08, J6 Bornier_5.08, J7 JST-XH, J8 JST-XH, J9 JST-XH, K1 SRD-05VDC-SL-C, K2 SRD-05VDC-SL-C, K3 SRD-05VDC-SL-C, K4 SRD-05VDC-SL-C, K5 SRD-05VDC-SL-C, K6 SRD-05VDC-SL-C, Q1 BC337-40, Q10 BC337-40, Q11 NDP6020P, Q2 BC337-40, Q3 BC337-40, Q4 BC337-40, Q5 BC337-40, Q6 BC337-40, Q7 NDP6020P, Q8 BC337-40, Q9 BS250

Commit message: [n3-universal] rev 0.1.2 : Q11 IRF4905 + zener D9, RV1 empreinte disque, trou nylon H5, serigraphie
- Q11 NDP6020P (VGS max +/-8 V) remplace par IRF4905PBF (VGS +/-20 V) : VGS = -VBAT en profil bus 12 V
- D9 1N4744A (15 V) grille-source de Q11, R40 limite son courant
- RV1 sur RV_Disc_D12mm_W5.4mm_P7.5mm (GEN-04), trou H5 vis nylon au coin secteur (GEN-05)
- serigraphie : JACK 5V, I2C J21/J22, polarites J18/J19/J25
- finalize_board : synchro empreintes/valeurs/descriptions + pistes D9
- table LCSC nettoyee des codes faux (C72503, C9135, C293822)
- DRC 0 erreur / 0 non connecte / 0 ecart de parite ; gerbers v0.1.2 (v0.1.1 retire)

Co-authored-by: Cursor <cursoragent@cursor.com>
Parts:
- added D9: 1N4744A, n3u:D_DO-41_SOD81_P5.08mm_Vertical_AnodeUp, F.Cu at (237.1, 150.5)
- added H5: M3, n3u:MountingHole_3.2mm_M3, F.Cu at (275.5, 59.0)
- Q11: value NDP6020P -> IRF4905
- RV1: footprint n3u:CP_Radial_D10.0mm_P5.00mm -> n3u:RV_Disc_D12mm_W5.4mm_P7.5mm
- moved RV1 2.24 mm to (252.0, 60.0)
Routing:
- net VBAT12_PROT: track 45.5 -> 50.0 mm
- net QP_G: track 18.8 -> 23.3 mm
- net MAINS_N: track 64.1 -> 62.5 mm
- net MAINS_LF: track 67.5 -> 66.3 mm
Other:
- board text added: "H5=NYLON"
- board text added: "I2C J21/J22"
- board text added: "JACK 5V"
- board text added: "n3-universal v0.1.2 — msp / n3pp / ffp5cs"
- board text removed: "5V 3A"
- board text removed: "I2C EXT x3"
- board text removed: "n3-universal v0.1.1 — msp / n3pp / ffp5cs"

Commit message: [n3-universal] rev 0.2 (WIP) : régénération complète — alim, cavaliers, borniers à vis, gardes
Point d'étape avant la fin du routage (freerouting en cours, 5 liaisons à
reprendre à la main) ; le PCB committé ici est intermédiaire.

generate.py 0.2 : rail capteurs Q7 IRF4905 + U1 LD1117V33 (JP1 bypass),
pont VBAT permanent (R38 + JP12 22k/100k, R49/C13, clamp D11 sur empreinte
double DO-35/SOD-123), Q12 IRF4905 anti-inversion + D12 1.5KE6.8A sur l'entrée
5 V, D8 1.5KE18A, cavaliers de forçage JP5-JP10 (K3 sans ON) + R61-R66, header
J38 CMD SENSE, borniers à vis 5,08 partout (bornier-4 HC-SR04), JP11 SD MISO,
diviseurs ADC/US par cavaliers JP13-JP21, TO-92 pas 2,54, TP1-4, 7 trous M3,
fusible sur empreinte universelle (clips 22,5 ou BLX-A 22,0), règle DRU
mains_creepage 6,4 mm, empilage 2 oz HAL sans plomb, SOURCING (Maroc / colis
LCSC, codes vérifiés le 2026-10-06), garde de recouvrement des étiquettes du
schéma, champ Description sur les empreintes (parité KiCad 10).

route_universal.py : API KiCad 10, retrait des pads A' avant chargement,
ponts A/A' du DevKit, keepouts COM resserrés, fentes COM allongées y66-83.
tidy_silkscreen.py : interdit d'entrer dans le courtyard d'un autre composant.
tools : check_silk_refs.py (nouveau, en CI), check_pcb_clearance.py
(bornier-4, couloirs USB avec offset), check_pinmap_vs_firmware.py (topologies
0.2). export_pcba.py : BOM/CPL PCBA dérivés de BOM.csv + CPL.
finalize_board.py : obsolète (garde-fou à l'exécution).

Docs : README (tableau 0.1.2 → 0.2, cavaliers), COMMANDE.md (JLCPCB, colis
d'import, achats Maroc), EVOLUTIONS_PROPOSEES (décisions actées), audit §14
(squelette), COMPOSANTS_FFP5CS.csv, hardware/README, COMMANDE_JLCPCB,
VERIFICATION, TUTO_PCB §4.bis.

Sources : empreintes dérivées de kicad-footprints (CC-BY-SA 4.0,
https://gitlab.com/kicad/libraries/kicad-footprints) ; freerouting 2.1.0
(https://github.com/freerouting/freerouting, GPL-3.0, outil non embarqué) ;
fiches ST LD1117, Infineon IRF4905, Littelfuse 1.5KE, Xuc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
Parts:
- removed Q10: BC337-40, n3u:TO-92_Inline
- removed Q9: BS250, n3u:TO-92_Inline
- removed R36, R37: 100k, n3u:R_Axial_DIN0207_L6.3mm_D2.5mm_P10.16mm_Horizontal
- added C10: 100n, n3u:C_Disc_D5.0mm_W2.5mm_P5.00mm, F.Cu at (217.0, 149.0)
- added C11: 10u/25V, n3u:CP_Radial_D5.0mm_P2.50mm, F.Cu at (226.0, 122.0)
- added C12: 100u/16V, n3u:CP_Radial_D6.3mm_P2.50mm, F.Cu at (235.0, 122.0)
- added C13: 100n, n3u:C_Disc_D5.0mm_W2.5mm_P5.00mm, F.Cu at (161.0, 122.0)
- added C6: 100n, n3u:C_Disc_D5.0mm_W2.5mm_P5.00mm, F.Cu at (132.0, 149.0)
- added C7: 100n, n3u:C_Disc_D5.0mm_W2.5mm_P5.00mm, F.Cu at (153.0, 149.0)
- added C8: 100n, n3u:C_Disc_D5.0mm_W2.5mm_P5.00mm, F.Cu at (174.0, 149.0)
- added C9: 100n, n3u:C_Disc_D5.0mm_W2.5mm_P5.00mm, F.Cu at (195.0, 149.0)
- added D11: BAT85, n3u:D_DO-35_SOD-123_Dual_P7.62mm, F.Cu at (171.0, 122.0)
- added D12: 1.5KE6.8A, n3u:D_DO-201AD_P15.24mm_Horizontal, F.Cu at (56.0, 114.0)
- added H6: M3, n3u:MountingHole_3.2mm_M3, F.Cu at (165.0, 153.0)
- added H7: M3, n3u:MountingHole_3.2mm_M3, F.Cu at (235.0, 153.0)
- added J38: Header CMD SENSE, n3u:PinHeader_1x08_P2.54mm_Vertical, F.Cu at (133.0, 154.0)
- added JP10: Jumper ON/OFF, n3u:PinHeader_1x03_P2.54mm_Vertical, F.Cu at (248.5, 90.0)
- added JP11: Jumper SD MISO, n3u:PinHeader_1x03_P2.54mm_Vertical, F.Cu at (209.0, 130.0)
- added JP12: Jumper profil, n3u:PinHeader_1x03_P2.54mm_Vertical, F.Cu at (133.0, 122.0)
- added JP13: Jumper profil, n3u:PinHeader_1x02_P2.54mm_Vertical, F.Cu at (147.0, 111.0)
- added JP14: Jumper profil, n3u:PinHeader_1x02_P2.54mm_Vertical, F.Cu at (168.0, 111.0)
- added JP15: Jumper profil, n3u:PinHeader_1x02_P2.54mm_Vertical, F.Cu at (189.0, 111.0)
- added JP16: Jumper profil, n3u:PinHeader_1x02_P2.54mm_Vertical, F.Cu at (147.0, 139.0)
- added JP17: Jumper profil, n3u:PinHeader_1x02_P2.54mm_Vertical, F.Cu at (168.0, 139.0)
- added JP18: Jumper profil, n3u:PinHeader_1x02_P2.54mm_Vertical, F.Cu at (189.0, 139.0)
- added JP19: Jumper profil, n3u:PinHeader_1x02_P2.54mm_Vertical, F.Cu at (210.0, 139.0)
- added JP20: Jumper profil, n3u:PinHeader_1x02_P2.54mm_Vertical, F.Cu at (232.0, 139.0)
- added JP21: Jumper profil, n3u:PinHeader_1x02_P2.54mm_Vertical, F.Cu at (211.0, 111.0)
- added JP5: Jumper ON/OFF, n3u:PinHeader_1x03_P2.54mm_Vertical, F.Cu at (78.5, 90.0)
- added JP6: Jumper ON/OFF, n3u:PinHeader_1x03_P2.54mm_Vertical, F.Cu at (112.5, 90.0)
- added JP7: Jumper ON/OFF, n3u:PinHeader_1x03_P2.54mm_Vertical, F.Cu at (146.5, 90.0)
- added JP8: Jumper ON/OFF, n3u:PinHeader_1x03_P2.54mm_Vertical, F.Cu at (180.5, 90.0)
- added JP9: Jumper ON/OFF, n3u:PinHeader_1x03_P2.54mm_Vertical, F.Cu at (214.5, 90.0)
- added Q12: IRF4905, n3u:TO-220-3_Vertical_GDS, F.Cu at (58.0, 106.0)
- added R48: 10k, n3u:R_Axial_DIN0207_L6.3mm_D2.5mm_P10.16mm_Horizontal, F.Cu at (210.0, 116.0)
- added R49: 1k, n3u:R_Axial_DIN0207_L6.3mm_D2.5mm_P10.16mm_Horizontal, F.Cu at (147.0, 122.0)
- added R50: 1k, n3u:R_Axial_DIN0207_L6.3mm_D2.5mm_P10.16mm_Horizontal, F.Cu at (132.0, 144.0)
- added R51: 1k, n3u:R_Axial_DIN0207_L6.3mm_D2.5mm_P10.16mm_Horizontal, F.Cu at (153.0, 144.0)
- added R52: 1k, n3u:R_Axial_DIN0207_L6.3mm_D2.5mm_P10.16mm_Horizontal, F.Cu at (174.0, 144.0)
- added R53: 1k, n3u:R_Axial_DIN0207_L6.3mm_D2.5mm_P10.16mm_Horizontal, F.Cu at (195.0, 144.0)
- added R54: 1k, n3u:R_Axial_DIN0207_L6.3mm_D2.5mm_P10.16mm_Horizontal, F.Cu at (217.0, 144.0)
- added R57: 100k, n3u:R_Axial_DIN0207_L6.3mm_D2.5mm_P10.16mm_Horizontal, F.Cu at (68.0, 108.0)
- added R58: 100k, n3u:R_Axial_DIN0207_L6.3mm_D2.5mm_P10.16mm_Horizontal, F.Cu at (174.0, 116.0)
- added R61: 1k, n3u:R_Axial_DIN0207_L6.3mm_D2.5mm_P10.16mm_Horizontal, F.Cu at (74.0, 89.3)
- added R62: 1k, n3u:R_Axial_DIN0207_L6.3mm_D2.5mm_P10.16mm_Horizontal, F.Cu at (108.0, 89.3)
- added R64: 1k, n3u:R_Axial_DIN0207_L6.3mm_D2.5mm_P10.16mm_Horizontal, F.Cu at (176.0, 89.3)
- added R65: 1k, n3u:R_Axial_DIN0207_L6.3mm_D2.5mm_P10.16mm_Horizontal, F.Cu at (210.0, 89.3)
- added R66: 1k, n3u:R_Axial_DIN0207_L6.3mm_D2.5mm_P10.16mm_Horizontal, F.Cu at (244.0, 89.3)
- added TP1: GND, n3u:TestPoint_THTPad_D2.0mm_Drill1.0mm, F.Cu at (224.0, 131.0)
- added TP2: +5V, n3u:TestPoint_THTPad_D2.0mm_Drill1.0mm, F.Cu at (228.0, 131.0)
- added TP3: +3V3_SW, n3u:TestPoint_THTPad_D2.0mm_Drill1.0mm, F.Cu at (232.0, 131.0)
- added TP4: +3V3, n3u:TestPoint_THTPad_D2.0mm_Drill1.0mm, F.Cu at (236.0, 131.0)
- added U1: LD1117V33, n3u:TO-220-3_Vertical_LDO, F.Cu at (214.0, 122.0)
- D8: value P6KE18A -> 1.5KE18A
- F1: footprint n3u:Fuse_5x20_Horizontal -> n3u:Fuse_5x20_Universal
- J10, J29, J30: value JST-XH -> Bornier_5.08; footprint n3u:JST_XH_B3B-XH-A_1x03_P2.50mm_Vertical -> n3u:TerminalBlock_bornier-3_P5.08mm
- J7, J8, J9: value JST-XH -> Bornier_5.08; footprint n3u:JST_XH_B4B-XH-A_1x04_P2.50mm_Vertical -> n3u:TerminalBlock_bornier-4_P5.08mm
- Q1, Q2, Q3, Q4, Q5, Q6, Q8: footprint n3u:TO-92_Inline -> n3u:TO-92_Inline_Wide_CBE
- Q11: footprint n3u:TO-220-3_Vertical -> n3u:TO-220-3_Vertical_GDS
- Q7: value NDP6020P -> IRF4905; footprint n3u:TO-220-3_Vertical -> n3u:TO-220-3_Vertical_GDS
- R17, R18, R19: value 2k* -> 2k
- R27, R43, R44, R45, R46, R47: value 10k* -> 10k
- R38: value 100k* -> 100k
- R39: value 22k* -> 22k
- RV1: value 10D471K -> 14D471K; footprint n3u:RV_Disc_D12mm_W5.4mm_P7.5mm -> n3u:RV_Disc_D15.5mm_W8mm_P7.5mm
- moved R27 135.0 mm to (217.0, 139.0)
- moved J10 97.2 mm to (86.0, 166.0)
- moved R43 88.1 mm to (132.0, 139.0)
- moved R26 82.0 mm to (210.0, 106.0)
- moved C3 74.4 mm to (238.0, 106.0)
- moved R25 67.5 mm to (196.0, 106.0)
- moved R44 66.6 mm to (153.0, 139.0)
- moved J29 58.5 mm to (53.0, 166.0)
- moved R23 55.8 mm to (224.0, 106.0)
- moved J30 55.1 mm to (69.5, 166.0)
- moved R38 54.0 mm to (132.0, 116.0)
- moved J31 52.2 mm to (190.0, 166.0)
- moved J32 49.8 mm to (206.5, 166.0)
- moved R39 49.0 mm to (153.0, 116.0)
- moved J33 47.4 mm to (223.0, 166.0)
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Connections:
- A1 pad 19: SD_MISO -> SD_MISO_W
- A2 pad 20: SD_MISO -> SD_MISO_S3
- J1 pad 1: +5V -> VIN_RAW
- J12 pad 2: ADC_E -> ADC_E_IN
- J2 pad 1: +5V -> VIN_RAW
- J31 pad 2: ADC_A -> ADC_A_IN
- J32 pad 2: ADC_B -> ADC_B_IN
- J33 pad 2: ADC_C -> ADC_C_IN
- J34 pad 2: ADC_D -> ADC_D_IN
- J37 pad 1: +5V -> VIN_RAW
- JP1 pad 1: +3V3 -> +5V
- JP1 pad 2: +3V3_SW -> LDO_IN
- Q7 pad 2: +3V3_SW -> +5V
- Q7 pad 3: +3V3 -> LDO_IN
- R17 pad 2: GND -> US_AQUA_DIV
- R18 pad 2: GND -> US_TANK_DIV
- R19 pad 2: GND -> US_POTA_DIV
- R27 pad 1: ADC_E -> ADC_E_IN
- R27 pad 2: GND -> ADC_E_DIV
- R35 pad 1: +3V3 -> +5V
- R38 pad 1: VBAT_SW -> VBAT_SENSE
- R38 pad 2: ADC_VBAT -> VBAT_DIV
- R39 pad 1: ADC_VBAT -> VBAT_22K
- R43 pad 1: ADC_A -> ADC_A_IN
- R43 pad 2: GND -> ADC_A_DIV
- R44 pad 1: ADC_B -> ADC_B_IN
- R44 pad 2: GND -> ADC_B_DIV
- R45 pad 1: ADC_C -> ADC_C_IN
- R45 pad 2: GND -> ADC_C_DIV
- R46 pad 1: ADC_D -> ADC_D_IN
- R46 pad 2: GND -> ADC_D_DIV
- R47 pad 2: US2 -> DHT_EXT_PU
Routing:
- net GND: track 930.1 -> 1346.2 mm, vias 46 -> 39
- net VIN_RAW: track 0.00 -> 301.5 mm, vias 0 -> 2
- net ADC_E_IN: track 0.00 -> 182.3 mm
- net +3V3: track 252.1 -> 426.2 mm, vias 1 -> 4
- net REL6_SW: track 24.9 -> 170.2 mm, vias 0 -> 1
- net REL1_SW: track 24.9 -> 151.8 mm, vias 0 -> 1
- net SD_MISO: track 158.7 -> 32.1 mm
- net SD_MISO_W: track 0.00 -> 120.3 mm, vias 0 -> 2
- net REL5_SW: track 24.9 -> 143.7 mm, vias 0 -> 2
- net DHT_INT: track 176.6 -> 279.9 mm, vias 1 -> 6
- net SD_MISO_S3: track 0.00 -> 99.9 mm
- net GATE: track 182.9 -> 281.4 mm
- net I2C_SDA: track 276.1 -> 371.1 mm, vias 3 -> 6
- net ADC_A_IN: track 0.00 -> 93.8 mm, vias 0 -> 2
- net +3V3_SW: track 538.8 -> 625.9 mm
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Other:
- board size 278 x 120 mm -> 278 x 135 mm
- board text added: "!! 230V !!"
- board text added: "+5V"
- board text added: "--"
- board text added: "12V"
- board text added: "1S"
- board text added: "2-3=WROOM"
- board text added: "3V3 SW"
- board text added: "3V3SW"
- board text added: "5V GND 3V3SW"
- board text added: "5V IN"
- board text added: "5V OUT"
- board text added: "ADC"
- board text added: "ANTENNE S3 : pas de cuivre"
- board text added: "BUS 12V : FUSIBLE LAME 7,5-10A EN AMONT"
- board text added: "CMD SENSE"
- board text added: "CS"
- board text added: "DAT"
- board text added: "DATA"
- board text added: "DO"
- board text added: "DS3231"
- board text added: "ECHO"
- board text added: "G"
- board text added: "INA226"
- board text added: "JACK 5V C+"
- board text added: "JP1 BYPASS"
- board text added: "JP1 FERME = rail 3V3 permanent (ffp5cs)"
- board text added: "JP1 OUVERT = commute par GPIO13 (msp, n3pp)"
- board text added: "JP1 ferme, JP13-15 fermes"
- board text added: "JP12 2-3 (1S)"
- board text added: "JP16-19 + JP21 fermes"
- board text added: "JP16-20 FERME = LDR | OUVERT = sonde sol n3pp, module AO msp"
- board text added: "JP20 ferme, JP12 1-2 (12V)"
- board text added: "JP20 ferme, JP12 2-3 (1S)"
- board text added: "JP5-10 FORCAGE : sans cavalier=AUTO | 1-2 ON | 2-3 OFF"
- board text added: "K1 FORCE"
- board text added: "K2 FORCE"
- board text added: "K3 FORCE"
- board text added: "K4 FORCE"
- board text added: "K5 FORCE"
- board text added: "K6 FORCE"
- board text added: "MISO"
- board text added: "MOSI"
- board text added: "OFF"
- board text added: "ON"
- board text added: "P"
- board text added: "PROFIL ffp5cs :"
- board text added: "PROFIL msp : JP1 ote,"
- board text added: "PROFIL n3pp : JP1 ote,"
- board text added: "SCK"
- board text added: "SD 1-2=S3"
- board text added: "SD : 1-2 = S3, 2-3 = WROOM"
- board text added: "SERVICE"
- board text added: "SIG"
- board text added: "TRIG"
- board text added: "US ECHO : JP13-15 = ffp5cs"
- board text added: "VBAT"
- board text added: "ZONE 230V - DANGER - COUPER LE SECTEUR AVANT INTERVENTION"
- board text added: "autres JP : OUVERTS"
- board text added: "ffp5cs"
- board text added: "msp"
- board text added: "n3-universal v0.2 — msp / n3pp / ffp5cs"
- board text removed: "!! ZONE 230V - DANGER !!"
- board text removed: "ALIM"
- board text removed: "ANTENNE : pas de cuivre dessous"
- board text removed: "ANTENNE S3: zone degagee"
- board text removed: "BUS 12V: FUSIBLE LAME 7,5-10A EN AMONT OBLIGATOIRE"
- board text removed: "COUPER LE SECTEUR AVANT INTERVENTION"
- board text removed: "GATE +3V3_SW (GPIO13)"
- board text removed: "GPIO"
- board text removed: "HC-SR04 : R17-R19 REQUISES (ffp5cs)"
- board text removed: "I2C EXT x2 + INA/DS3231"
- board text removed: "J20 5V/GND/3V3SW"
- board text removed: "JACK 5V"
- board text removed: "JP SD 1-2=S3 2-3=WROOM"
- board text removed: "JP1 FERME=permanent ffp5cs / OUVERT=msp,n3pp"
- board text removed: "JP1: FERME=ffp5cs"
- board text removed: "LDR msp (R pose) / SONDE SOL n3pp (sans R)"
- board text removed: "PONT DIV VBAT (R38/R39 selon profil)"
- board text removed: "SD"
- board text removed: "SRV GROS"
- board text removed: "SRV PETITS"
- board text removed: "n3-universal v0.1.2 — msp / n3pp / ffp5cs"

Commit message: [n3-universal] rev 0.2 : routage complet, sérigraphie, exports 2 oz, docs, garde PCBA
PCB 0.2 routé et vérifié (KiCad 10.0.6, freerouting 2.1.0) : DRC 0 erreur,
0 non connecté, 0 écart de parité avec les règles clearance 3 mm, creepage
6,4 mm et plans 6,5 mm ; écart secteur/logique 3 mm : 0 violation, plan GND
à 6,50 mm du secteur ; 62 avertissements de sérigraphie (contours des
relais/PSU sur les fentes, libellé « C » de Q8 sur le contour de C12).
Pinmap, corps 3D/couloirs, repères, rôles : OK.

Routage : 3 instances freerouting en parallèle puis itérations sur le
câblage existant (route_universal.py --ses / --dsn-only, DSN avec le
câblage) jusqu'à 0 liaison logique non routée ; vias de couture hors corps
et hors étiquettes ; stubs pendants retirés (cleanup piloté par le DRC).

Sérigraphie : tidy_silkscreen interdit d'entrer dans le courtyard d'un
voisin, tolère un via tenté en repli, garde le repère à <= 3 mm du corps
(même mesure que tools/check_silk_refs.py) ; repères TO-92/TO-220/headers/
TP/bornier-4 repositionnés, légendes (forçage, modules, NYLON) replacées,
libellés CS/SCK/MOSI/MISO abandonnés (pas de place : JP2/3/4/11 + README),
valeurs R35/R48 dégagées de Q7/U1, D11 « K » et libellés TO-220 à 0,8 mm.

Exports : gerbers-n3-universal-v0.2.zip (10 fichiers, gbrjob 2 oz, DRC
bloquant), schéma PDF, SVG, rendu 3D, BOM/CPL JLCPCB et NextPCB,
exports/pcba/ dérivés par export_pcba.py (42 groupes / 154 pièces du socle,
11 conditionnelles profils secteur et bus 12 V). Zip 0.1.2 retiré.

Docs : README (état 0.2, cavaliers : sans cavalier = AUTO, 1-2 = ON,
2-3 = OFF), audit §14 (contrôles, approvisionnement LCSC vérifié, risques
résiduels), COMMANDE.md, EVOLUTIONS_PROPOSEES, TUTO_PCB §4.bis,
exports/pcba/README. ~*.lck ignorés.

Sources : kicad-footprints (CC-BY-SA 4.0,
https://gitlab.com/kicad/libraries/kicad-footprints) ; freerouting v2.1.0
(https://github.com/freerouting/freerouting, GPL-3.0, outil non embarqué).

Co-Authored-By: Claude Fable 5.1 <noreply@anthropi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
Routing:
- net I2C_SCL: track 257.6 -> 359.4 mm, vias 4 -> 3
- net SD_MOSI_S3: track 7.70 -> 105.5 mm
- net REL2_SW: track 31.4 -> 126.7 mm, vias 0 -> 1
- net US3: track 169.8 -> 263.1 mm, vias 1 -> 2
- net K3: track 204.1 -> 273.1 mm, vias 3 -> 2
- net SPARE_TX0: track 221.2 -> 282.2 mm, vias 1 -> 5
- net GATE: track 281.4 -> 231.2 mm, vias 5 -> 4
- net +5V: track 760.1 -> 808.6 mm, vias 3 -> 1
- net REL6_SW: track 170.2 -> 209.8 mm, vias 1 -> 4
- net K1: track 272.2 -> 308.2 mm, vias 3 -> 4
- net +3V3_SW: track 625.9 -> 599.1 mm, vias 0 -> 1
- net ADC_VBAT: track 211.5 -> 186.1 mm, vias 4 -> 0
- net I2C_SDA: track 371.1 -> 346.5 mm, vias 6 -> 2
- net DHT_INT: track 279.9 -> 255.9 mm, vias 6 -> 5
- net GND: track 1346.2 -> 1322.8 mm, vias 39 -> 14
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Other:
- board text added: "JP5-10 : rien = AUTO 1-2 = ON 2-3 = OFF"
- board text added: "NYLON"
- board text added: "UN SEUL MODULE : A1 OU A2"
- board text removed: "CS"
- board text removed: "H5=NYLON"
- board text removed: "JP1 BYPASS"
- board text removed: "JP5-10 FORCAGE : sans cavalier=AUTO | 1-2 ON | 2-3 OFF"
- board text removed: "MISO"
- board text removed: "MOSI"
- board text removed: "SCK"
- board text removed: "SD : 1-2 = S3, 2-3 = WROOM"
- board text removed: "UN SEUL MODULE : A1 (WROOM) OU A2 (S3)"
