File: hardware/n3-universal/kicad/n3-universal.kicad_sch (KiCad schematic)
At the start: 127 parts, among them J1 Bornier_5.08, J10 JST-XH, J11 Bornier_5.08, J12 Bornier_5.08, J13 Support OLED, J14 Support I2C ext, J15 Header servo, J16 Header servo, J17 Header service, J18 Bornier_5.08, J19 Bornier_5.08, J2 Jack 5.5/2.1, J20 Header alim, J21 Support I2C libre, J22 Support I2C libre, J23 Bornier_5.08, J24 Bornier_5.08, J25 Bornier_5.08, J26 Bornier_5.08, J27 Bornier_5.08, J28 Support I2C libre, J29 JST-XH, J3 Bornier_5.08, J30 JST-XH, J31 Bornier_5.08, J32 Bornier_5.08, J33 Bornier_5.08, J34 Bornier_5.08, J35 Support module microSD, J36 Bornier_5.08, J37 Bornier_5.08, J4 Bornier_5.08, J5 Bornier_5.08, J6 Bornier_5.08, J7 JST-XH, J8 JST-XH, J9 JST-XH, K1 SRD-05VDC-SL-C, K2 SRD-05VDC-SL-C, K3 SRD-05VDC-SL-C, K4 SRD-05VDC-SL-C, K5 SRD-05VDC-SL-C, K6 SRD-05VDC-SL-C, Q1 BC337-40, Q10 BC337-40, Q11 NDP6020P, Q2 BC337-40, Q3 BC337-40, Q4 BC337-40, Q5 BC337-40, Q6 BC337-40, Q7 NDP6020P, Q8 BC337-40, Q9 BS250

Commit message: fix(n3-universal): géométrie secteur sans croisement, contour réparé, passe de placement complète
PSU : J27/F1/RV1 hors du corps du Hi-Link (décalé à x303), pistes L/N/LF
redessinées sans croisement ni court (varistance re-câblée N/LF), fente
frontière y71-73 disjointe de la fente verticale (contour valide). ~30
repositionnements sur courtyards réels (rangée basse de borniers y151,
colonne gate/diviseur/SD décalée hors des canaux relais 5/6 et du bloc DHT,
servos/J17/J20 rive droite, trous de fixation déplacés hors zone secteur).
ERC 0 erreur, garde anti-dérive vert, 1 seul avertissement de recouvrement
résiduel corrigé. Routage v2 en cours.

Co-Authored-By: Claude <noreply@anthropic.com>
Claude-Session: https://claude.ai/code/session_01HcxShQb65yktRwp31wBq9q
Connections:
- net MAINS_LF: now also RV1.2; no longer RV1.1
- net MAINS_N: now also RV1.1; no longer RV1.2
Changed lines of the file:
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@@
   (wire (pts (xy 388.62 208.28) (xy 386.08 208.28))
     (stroke (width 0) (type default)))
-  (label "MAINS_LF" (at 386.08 208.28 0)
+  (label "MAINS_N" (at 386.08 208.28 0)
     (effects (font (size 1.27 1.27)) (justify right bottom))
 )
   (wire (pts (xy 398.78 208.28) (xy 401.32 208.28))
     (stroke (width 0) (type default)))
-  (label "MAINS_N" (at 401.32 208.28 0)
+  (label "MAINS_LF" (at 401.32 208.28 0)
     (effects (font (size 1.27 1.27)) (justify left bottom))
 )

Commit message: fix(n3-universal): corrections de l'audit final — Q11, coin PSU 230V, plan GND, H1, poses conditionnelles + contrats serveur (n3pp 4.72, ffp5cs 15.29)
Audit exhaustif multi-axes (netlist alim/signaux, strapping, géométrie secteur,
firmwares, contrats serveur) avant commande. Corrections carte (PCB routé,
schéma régénéré, générateur synchronisé, gerbers/PDF/SVG re-exportés — PTH 521) :

- Q11 (anti-inversion bus 12V) : câblé au brochage BS250 (D-G-S), l'entrée 12 V
  arrivait sur la GRILLE du NDP6020P (TO-220 : 1=G 2=D 3=S) — profil 12 V
  inopérant et Vgs hors spec. Recâblé G/D/S comme Q7 ; liaisons re-routées B.Cu.
- Coin PSU 230 V re-routé : L passait à 0,75 mm du pad neutre de J27 (tronçon
  non fusé), N // LF à 1,5 mm. Nouveau tracé avec écarts L<->N<->LF >= 3 mm hors
  pas des composants ; J27 devient 1=N / 2=L, repères L/N sérigraphiés.
- Plan GND exclu du coin PSU (246..318 x 40..73, F+B) : il coulait sous les
  pistes/pads 230 V ; check_mains_gap voit désormais les ZONES REMPLIES
  (il était aveugle au cuivre coulé) — 0 violation.
- H1 (coin relais, enclavé par K1) : vis NYLON obligatoire (tête métal à
  ~4,3 mm du 230 V) — keepout de coulée sous la tête + sérigraphie H1=NYLON.
- Poses conditionnelles (BOM étoilée) : R17/R18/R19 (2k, ponts écho HC-SR04)
  posées ffp5cs uniquement — permanentes, elles verrouillaient PLUIE/US1 à
  « mouillé » et rendaient DHT_EXT/US2 illisible côté msp (niveau haut ~0,55 V) ;
  R27 (10k) posée pour LDR seulement (module AO msp atténué de moitié sinon).
- microSD/MTDI : module 3,3 V direct sans tampon, réservé S3 ; sur WROOM efuse
  VDD_SDIO=3V3 obligatoire (une carte SD peut tirer GPIO12 haut au boot).
  Étiquettes servo égarées en zone secteur repositionnées ; JP1 « 1-2 » précisé.

Contrats serveur (croisements découverts par l'audit) :
- n3pp v4.72 : clé JSON pompe découplée de la broche (POMPE_OUTPUT_KEY="12" —
  en universel POMPE=16 lisait une ligne legacy non exposée par l'UI).
- ffp5cs v15.29 : gpio_mapping.h reprend le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
Parts:
- Q11: symbol n3u:PMOS_DGS -> n3u:PMOS_GDS
- R17, R18, R19: value 2k -> 2k*
- R27: value 10k -> 10k*
Connections:
- net MAINS_L: now also J27.2; no longer J27.1
- net MAINS_N: now also J27.1; no longer J27.2
- net QP_G: now also Q11.1 (G); no longer Q11.2 (G)
- net VBAT12_IN: now also Q11.2 (D); no longer Q11.1 (D)
Changed lines of the file:
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@@
     (exclude_from_sim no) (in_bom yes) (on_board yes) (dnp no)
     (property "Reference" "R17" (at 233.68 40.64 0) (effects (font (size 1.27 1.27))))
-    (property "Value" "2k" (at 233.68 42.78 0) (effects (font (size 1.27 1.27))))
+    (property "Value" "2k*" (at 233.68 42.78 0) (effects (font (size 1.27 1.27))))
     (property "Footprint" "n3u:R_Axial_DIN0207_L6.3mm_D2.5mm_P10.16mm_Horizontal" (at 233.68 45.72 0) (effects (font (size 1.27 1.27)) (hide yes)))
     (property "Datasheet" "~" (at 233.68 45.72 0) (effects (font (size 1.27 1.27)) (hide yes)))
-    (property "Description" "Pont diviseur écho AQUA (5V->3V3)" (at 233.68 45.72 0) (effects (font (size 1.27 1.27)) (hide yes)))
+    (property "Description" "Pont diviseur écho AQUA (5V->3V3) — POSER pour ffp5cs ; ABSENT sur unités msp (et R19 absent si option wroom-sd)" (at 233.68 45.72 0) (effects (font (size 1.27 1.27)) (hide yes)))
     (pin "1")
     (pin "2")
@@
     (exclude_from_sim no) (in_bom yes) (on_board yes) (dnp no)
     (property "Reference" "R18" (at 233.68 71.12 0) (effects (font (size 1.27 1.27))))
-    (property "Value" "2k" (at 233.68 73.26 0) (effects (font (size 1.27 1.27))))
+    (property "Value" "2k*" (at 233.68 73.26 0) (effects (font (size 1.27 1.27))))
     (property "Footprint" "n3u:R_Axial_DIN0207_L6.3mm_D2.5mm_P10.16mm_Horizontal" (at 233.68 76.20 0) (effects (font (size 1.27 1.27)) (hide yes)))
     (property "Datasheet" "~" (at 233.68 76.20 0) (effects (font (size 1.27 1.27)) (hide yes)))
-    (property "Description" "Pont diviseur écho TANK (5V->3V3)" (at 233.68 76.20 0) (effects (font (size 1.27 1.27)) (hide yes)))
+    (property "Description" "Pont diviseur écho TANK (5V->3V3) — POSER pour ffp5cs ; ABSENT sur unités msp (et R19 absent si option wroom-sd)" (at 233.68 76.20 0) (effects (font (size 1.27 1.27)) (hide yes)))
     (pin "1")
     (pin "2")
@@
     (exclude_from_sim no) (in_bom yes) (on_board yes) (dnp no)
     (property "Reference" "R19" (at 233.68 101.60 0) (effects (font (size 1.27 1.27))))
-    (property "Value" "2k" (at 233.68 103.74 0) (effects (font (size 1.27 1.27))))
+    (property "Value" "2k*" (at 233.68 103.74 0) (effects (font (size 1.27 1.27))))
     (property "Footprint" "n3u:R_Axial_DIN0207_L6.3mm_D2.5mm_P10.16mm_Horizontal" (at 233.68 106.68 0) (effects (font (size 1.27 1.27)) (hide yes)))
     (property "Datasheet" "~" (at 233.68 106.68 0) (effects (font (size 1.27 1.27)) (hide yes)))
-    (property "Description" "Pont diviseur écho POTA (5V->3V3)" (at 233.68 106.68 0) (effects (font (size 1.27 1.27)) (hide yes)))
+    (property "Description" "Pont diviseur écho POTA (5V->3V3) — POSER pour ffp5cs ; ABSENT sur unités msp (et R19 absent si option wroom-sd)" (at 233.68 106.68 0) (effects (font (size 1.27 1.27)) (hide yes)))
     (pin "1")
     (pin "2")
@@
     (exclude_from_sim no) (in_bom yes) (on_board yes) (dnp no)
     (property "Reference" "R27" (at 233.68 182.88 0) (effects (font (size 1.27 1.27))))
-    (property "Value" "10k" (at 233.68 185.02 0) (effects (font (size 1.27 1.27))))
+    (property "Value" "10k*" (at 233.68 185.02 0) (effects (font (size 1.27 1.27))))
     (property "Footprint" "n3u:R_Axial_DIN0207_L6.3mm_D2.5mm_P10.16mm_Horizontal" (at 233.68 187.96 0) (effects (font (size 1.27 1.27)) (hide yes)))
     (property "Datasheet" "~" (at 233.68 187.96 0) (effects (font (size 1.27 1.27)) (hide yes)))
-    (property "Description" "Bas du pont diviseur LDR (GPIO34 = entrée seule ADC)" (at 233.68 187.96 0) (effects (font (size 1.27 1.27)) (hide yes)))
+    (property "Description" "Bas de pont LDR sur net ADC_E (GPIO36 WROOM / IO6 S3) — POSER pour LDR ; ABSENT pour module AO (msp HumiditeSol)" (at 233.68 187.96 0) (effects (font (size 1.27 1.27)) (hide yes)))
     (pin "1")
     (pin "2")
@@
     (effects (font (size 1.27 1.27)) (justify right bottom))
 )
-  (symbol (lib_id "n3u:PMOS_DGS") (at 393.70 132.08 0) (unit 1)
+  (symbol (lib_id "n3u:PMOS_GDS") (at 393.70 132.08 0) (unit 1)
     (exclude_from_sim no) (in_bom yes) (on_board yes) (dnp no)
     (property "Reference" "Q11" (at 393.70 124.46 0) (effects (font (size 1.27 1.27))))
@@
     (property "Footprint" "n3u:TO-220-3_Vertical" (at 393.70 132.08 0) (effects (font (size 1.27 1.27)) (hide yes)))
     (property "Datasheet" "~" (at 393.70 132.08 0) (effects (font (size 1.27 1.27)) (hide yes)))
-    (property "Description" "Anti-inversion P-MOSFET (1=D=entrée 2=G 3=S=sortie)" (at 393.70 132.08 0) (effects (font (size 1.27 1.27)) (hide yes)))
-    (pin "2")
-    (pin "1")
+    (property "Description" "Anti-inversion P-MOSFET (1=G 2=D=entrée 3=S=sortie)" (at 393.70 132.08 0) (effects (font (size 1.27 1.27)) (hide yes)))
+    (pin "1")
+    (pin "2")
     (pin "3")
     (instances (project "n3-universal" (path "/e48da96c-ccf9-5077-8ed8-2811f4041ce3" (reference "Q11") (unit 1))))
@@
     (property "Footprint" "n3u:TerminalBlock_bornier-2_P5.08mm" (at 370.84 198.12 0) (effects (font (size 1.27 1.27)) (hide yes)))
     (property "Datasheet" "~" (at 370.84 198.12 0) (effects (font (size 1.27 1.27)) (hide yes)))
-    (property "Description" "ENTREE SECTEUR 230V (1=L 2=N) — ZONE DANGER" (at 370.84 198.12 0) (effects (font (size 1.27 1.27)) (hide yes)))
+    (property "Description" "ENTREE SECTEUR 230V (1=N 2=L) — ZONE DANGER" (at 370.84 198.12 0) (effects (font (size 1.27 1.27)) (hide yes)))
     (pin "1")
     (pin "2")
@@
   (wire (pts (xy 364.49 195.58) (xy 361.95 195.58))
     (stroke (width 0) (type default)))
-  (label "MAINS_L" (at 361.95 195.58 0)
+  (label "MAINS_N" (at 361.95 195.58 0)
     (effects (font (size 1.27 1.27)) (justify right bottom))
 )
   (wire (pts (xy 364.49 198.12) (xy 361.95 198.12))
     (stroke (width 0) (type default)))
-  (label "MAINS_N" (at 361.95 198.12 0)
-    (effects (font (size 1.27 1.27)) (justify right bottom))
-)
+  (label "MAINS_L" (at 361.95 198.12 0)
+    (effects (font (size 1.27 1.27)) (justify right bottom))
+)

Commit message: docs(n3-universal): rapport d'audit pré-commande + corrections documentaires vérifiées
Consolide dans le dépôt les constats de l'audit du 2026-08-28 (7 dimensions,
verdict : commandable, 0 bloquant) et corrige les documents d'assemblage qui
contredisaient la carte. Aucune modification du PCB routé, des gerbers ni de
la netlist.

- AUDIT-2026-08-28.md : conformité vérifiée, 3 actions avant paiement (sourcing
  NDP6020P, mesure des entraxes HLK-20M05, cuivre 2 oz à cocher), constats
  retenus par sévérité, check-list rev 0.2.
- generate.py : textes du schéma remis sur la carte réelle — 6 canaux relais et
  leurs GPIO des deux sites (au lieu de 4 canaux aux GPIO de l'ancienne carte
  ffp5cs), servos sur SERVO1/SERVO2, LDR sur ADC_E, contenu réel du header J17,
  suppression de la référence à une résistance R22 inexistante ; en-tête et
  cartouche remis sur n3-universal ; cote réelle des relais SRD Form C
  (7 A/240 VAC, 3 A inductif) et note de pose de RV1 ; ajout des clips de
  porte-fusible, des cavaliers et de la visserie nylon de H1, jusque-là absents
  de la BOM alors qu'ils sont indispensables au montage.
- BOM.csv et kicad_sch régénérés via gen_bom()/gen_schematic() seuls — jamais
  main(), qui réécrirait un PCB non routé. Diff du schéma limité aux lignes
  text/Description/comment ; checker anti-dérive toujours vert.
- README : consigne boost 5 V du profil batterie 1S, frontière secteur exacte,
  vérification de l'ordre des broches des modules, dépeuplement de R28/R31 avant
  l'option wroom-sd, renvois vers COMMANDE.md et le rapport d'audit.
- check_pinmap_vs_firmware.py : docstring (UART0 réservé au header service).

exports/schema.pdf reste à ré-exporter sur un poste avec KiCad (export_fab.py).

Co-Authored-By: Claude Fable 5 <noreply@anthropic.com>
Claude-Session: https://claude.ai/code/session_01YUakdFj87xCernvTeSv8Rb
Other:
- note added: "6 RELAIS K1..K6 — commande ACTIVE HAUT (base 1k + pull-down 10k : etat sur au boot). WROOM : GPIO16/17/18/19/23/25 — S3 : IO15/16/17/18/48/45. Le role de chaque canal depend du firmware (voir les sections PINMAP_UNIVERSAL). Borniers : 1=NC 2=COM 3=NO. SRD Form C = 7A/240VAC et 3A inductif REELS par contact (le 10A ne vaut qu'en 125VAC ou en Form A). ZONE SECTEUR ISOLEE sur le PCB (fentes + 3mm mi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"
- note added: "HEADER SERVICE J17 : 3V3 / GND / EN / RX0 / TX0 / +5V uniquement. Tous les autres GPIO sont consommes par la carte universelle (GPIO36 = ADC_E, GPIO39 = ADC_VBAT). Laisser RX0/TX0 libres pendant le flash USB."
- note added: "LUMIERE : LDR déportée sur J12, net ADC_E (GPIO36 WROOM / IO6 S3). Bas de pont R27 10k : A POSER pour une LDR, ABSENT pour un module à sortie AO."
- note added: "SERVOS 5V (nets SERVO1/SERVO2) — WROOM : GPIO26/27, S3 : IO21/IO47. Signal en série R20/R21 (220R). Alimentation prise directement sur le rail +5V."
- note added: "SITE A1 : ESP32 DevKit V1 (30 broches, socketé) — UN SEUL module peuplé (A1 OU A2). Envs carte universelle : msp/n3pp esp32dev_universal_test, ffp5cs wroom-universal-test. Sur une unité ffp5cs, ÔTER JP1 avant un flash UART (le pull-up R24 sur GPIO2 bloque le bootloader)."
- note removed: "4 RELAIS 230V 10A — commande ACTIVE HAUT (actuators.h : on() = HIGH). REL1=Pompe aquarium GPIO16, REL2=Pompe réservoir GPIO18, REL3=Chauffage GPIO2, REL4=Lumière GPIO15. Borniers : 1=NC 2=COM 3=NO. ZONE SECTEUR ISOLEE sur le PCB (fentes + 3mm mini) — circuit 230V A PROTEGER EN AMONT (fusible/disjoncteur) ; charges inductives : snubber cote charge."
- note removed: "ESP32 DevKit V1 (30 broches, socketé). Flash/monitor via l'USB du module (pio run -e wroom-prod -t upload)."
- note removed: "LUMIERE : LDR déportée + 10k (GPIO34 = entrée seule)."
- note removed: "SERVOS NOURRISSEURS 5V GPIO12 (strapping MTDI) : pull-down R22, signal série R20."
- note removed: "TOUS les GPIO libres sur header (Dupont), y compris RX0/TX0 (les laisser libres pendant le flash USB) et GPIO36/39 (entrees seules)."
Changed lines of the file:
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@@
     (rev "0.1")
     (company "salle aeree n3")
-    (comment 1 "Genere par hardware/ffp5cs-wroom-prod/generator/generate.py")
-    (comment 2 "Source de verite : ffp5cs/include/pins.h (BOARD_WROOM) via pinmap.json")
+    (comment 1 "Genere par hardware/n3-universal/generator/generate.py")
+    (comment 2 "Source de verite : pinmap_universel_propose.json + sections PINMAP_UNIVERSAL (msp / n3pp / ffp5cs)")
   )
   (symbol (lib_id "n3u:ESP32_DEVKIT_V1_30") (at 152.40 88.90 0) (unit 1)
@@
     (property "Footprint" "n3u:Relay_SPDT_SANYOU_SRD_Series_Form_C" (at 330.20 15.24 0) (effects (font (size 1.27 1.27)) (hide yes)))
     (property "Datasheet" "~" (at 330.20 15.24 0) (effects (font (size 1.27 1.27)) (hide yes)))
-    (property "Description" "Relais 5V SPDT 10A/250VAC (Songle/Sanyou SRD)" (at 330.20 15.24 0) (effects (font (size 1.27 1.27)) (hide yes)))
+    (property "Description" "Relais 5V SPDT Songle/Sanyou SRD Form C — 7A/240VAC et 3A inductif REELS par contact (le 10A ne vaut qu'en 125VAC ou en Form A)" (at 330.20 15.24 0) (effects (font (size 1.27 1.27)) (hide yes)))
     (pin "5")
     (pin "2")
@@
     (property "Footprint" "n3u:Relay_SPDT_SANYOU_SRD_Series_Form_C" (at 330.20 81.28 0) (effects (font (size 1.27 1.27)) (hide yes)))
     (property "Datasheet" "~" (at 330.20 81.28 0) (effects (font (size 1.27 1.27)) (hide yes)))
-    (property "Description" "Relais 5V SPDT 10A/250VAC (Songle/Sanyou SRD)" (at 330.20 81.28 0) (effects (font (size 1.27 1.27)) (hide yes)))
+    (property "Description" "Relais 5V SPDT Songle/Sanyou SRD Form C — 7A/240VAC et 3A inductif REELS par contact (le 10A ne vaut qu'en 125VAC ou en Form A)" (at 330.20 81.28 0) (effects (font (size 1.27 1.27)) (hide yes)))
     (pin "5")
     (pin "2")
@@
     (property "Footprint" "n3u:Relay_SPDT_SANYOU_SRD_Series_Form_C" (at 330.20 147.32 0) (effects (font (size 1.27 1.27)) (hide yes)))
     (property "Datasheet" "~" (at 330.20 147.32 0) (effects (font (size 1.27 1.27)) (hide yes)))
-    (property "Description" "Relais 5V SPDT 10A/250VAC (Songle/Sanyou SRD)" (at 330.20 147.32 0) (effects (font (size 1.27 1.27)) (hide yes)))
+    (property "Description" "Relais 5V SPDT Songle/Sanyou SRD Form C — 7A/240VAC et 3A inductif REELS par contact (le 10A ne vaut qu'en 125VAC ou en Form A)" (at 330.20 147.32 0) (effects (font (size 1.27 1.27)) (hide yes)))
     (pin "5")
     (pin "2")
@@
     (property "Footprint" "n3u:Relay_SPDT_SANYOU_SRD_Series_Form_C" (at 330.20 213.36 0) (effects (font (size 1.27 1.27)) (hide yes)))
     (property "Datasheet" "~" (at 330.20 213.36 0) (effects (font (size 1.27 1.27)) (hide yes)))
-    (property "Description" "Relais 5V SPDT 10A/250VAC (Songle/Sanyou SRD)" (at 330.20 213.36 0) (effects (font (size 1.27 1.27)) (hide yes)))
+    (property "Description" "Relais 5V SPDT Songle/Sanyou SRD Form C — 7A/240VAC et 3A inductif REELS par contact (le 10A ne vaut qu'en 125VAC ou en Form A)" (at 330.20 213.36 0) (effects (font (size 1.27 1.27)) (hide yes)))
     (pin "5")
     (pin "2")
@@
     (property "Footprint" "n3u:Relay_SPDT_SANYOU_SRD_Series_Form_C" (at 330.20 279.40 0) (effects (font (size 1.27 1.27)) (hide yes)))
     (property "Datasheet" "~" (at 330.20 279.40 0) (effects (font (size 1.27 1.27)) (hide yes)))
-    (property "Description" "Relais 5V SPDT 10A/250VAC (Songle/Sanyou SRD)" (at 330.20 279.40 0) (effects (font (size 1.27 1.27)) (hide yes)))
+    (property "Description" "Relais 5V SPDT Songle/Sanyou SRD Form C — 7A/240VAC et 3A inductif REELS par contact (le 10A ne vaut qu'en 125VAC ou en Form A)" (at 330.20 279.40 0) (effects (font (size 1.27 1.27)) (hide yes)))
     (pin "5")
     (pin "2")
@@
     (property "Footprint" "n3u:Relay_SPDT_SANYOU_SRD_Series_Form_C" (at 330.20 345.44 0) (effects (font (size 1.27 1.27)) (hide yes)))
     (property "Datasheet" "~" (at 330.20 345.44 0) (effects (font (size 1.27 1.27)) (hide yes)))
-    (property "Description" "Relais 5V SPDT 10A/250VAC (Songle/Sanyou SRD)" (at 330.20 345.44 0) (effects (font (size 1.27 1.27)) (hide yes)))
+    (property "Description" "Relais 5V SPDT Songle/Sanyou SRD Form C — 7A/240VAC et 3A inductif REELS par contact (le 10A ne vaut qu'en 125VAC ou en Form A)" (at 330.20 345.44 0) (effects (font (size 1.27 1.27)) (hide yes)))
     (pin "5")
     (pin "2")
@@
     (property "Footprint" "n3u:CP_Radial_D10.0mm_P5.00mm" (at 393.70 208.28 0) (effects (font (size 1.27 1.27)) (hide yes)))
     (property "Datasheet" "~" (at 393.70 208.28 0) (effects (font (size 1.27 1.27)) (hide yes)))
-    (property "Description" "Varistance 300VAC transitoires secteur" (at 393.70 208.28 0) (effects (font (size 1.27 1.27)) (hide yes)))
+    (property "Description" "Varistance 300VAC transitoires secteur — pattes à replier (pas réel 7,5 mm sur une empreinte 5,0 mm) : pose main, à exclure d'un assemblage machine ; le repère + de l'empreinte est sans objet" (at 393.70 208.28 0) (effects (font (size 1.27 1.27)) (hide yes)))
     (pin "1")
     (pin "2")
@@
   (text "ALIMENTATION 5V (3A recommandé) — jack OU bornier.\nD5 protège le rail si l'USB du DevKit est branché en même temps." (exclude_from_sim no) (at 45.72 30.48 0)
     (effects (font (size 1.7 1.7)) (justify left bottom)))
-  (text "ESP32 DevKit V1 (30 broches, socketé).\nFlash/monitor via l'USB du module (pio run -e wroom-prod -t upload)." (exclude_from_sim no) (at 132.08 60.96 0)
+  (text "SITE A1 : ESP32 DevKit V1 (30 broches, socketé) — UN SEUL module peuplé (A1 OU A2).\nEnvs carte universelle : msp/n3pp esp32dev_universal_test, ffp5cs wroom-universal-test.\nSur une unité ffp5cs, ÔTER JP1 avant un flash UART (le pull-up R24 sur GPIO2 bloque le bootloader)." (exclude_from_sim no) (at 132.08 60.96 0)
     (effects (font (size 1.7 1.7)) (justify left bottom)))
-  (text "SERVOS NOURRISSEURS 5V\nGPIO12 (strapping MTDI) : pull-down R22, signal série R20." (exclude_from_sim no) (at 111.76 127.00 0)
+  (text "SERVOS 5V (nets SERVO1/SERVO2) — WROOM : GPIO26/27, S3 : IO21/IO47.\nSignal en série R20/R21 (220R). Alimentation prise directement sur le rail +5V." (exclude_from_sim no) (at 111.76 127.00 0)
     (effects (font (size 1.7 1.7)) (justify left bottom)))
   (text "3x HC-SR04 (5V), mode mono-broche TRIG=ECHO (sensor_ultrasonic.cpp).\nEcho 5V ramené à 3V3 par pont 1k/2k sur chaque canal." (exclude_from_sim no) (at 218.44 25.40 0)
@@
   (text "EAU : DS18B20 (1-Wire, pull-up 4.7k)." (exclude_from_sim no) (at 218.44 154.94 0)
     (effects (font (size 1.7 1.7)) (justify left bottom)))
-  (text "LUMIERE : LDR déportée + 10k (GPIO34 = entrée seule)." (exclude_from_sim no) (at 218.44 180.34 0)
+  (text "LUMIERE : LDR déportée sur J12, net ADC_E (GPIO36 WROOM / IO6 S3).\nBas de pont R27 10k : A POSER pour une LDR, ABSENT pour un module à sortie AO." (exclude_from_sim no) (at 218.44 180.34 0)
     (effects (font (size 1.7 1.7)) (justify left bottom)))
   (text "I2C : OLED SSD1306 0x3C + header extension (DS3231 si besoin)." (exclude_from_sim no) (at 218.44 205.74 0)
     (effects (font (size 1.7 1.7)) (justify left bottom)))
-  (text "4 RELAIS 230V 10A — commande ACTIVE HAUT (actuators.h : on() = HIGH).\nREL1=Pompe aquarium GPIO16, REL2=Pompe réservoir GPIO18,\nREL3=Chauffage GPIO2, REL4=Lumière GPIO15. Borniers : 1=NC 2=COM 3=NO.\nZONE SECTEUR ISOLEE sur le PCB (fentes + 3mm mini) — circuit 230V\nA PROTEGER EN AMONT (fusible/disjoncteur) ; charges inductives : snubber cote charge." (exclude_from_sim no) (at 271.78 2.54 0)
+  (text "6 RELAIS K1..K6 — commande ACTIVE HAUT (base 1k + pull-down 10k : etat sur au boot).\nWROOM : GPIO16/17/18/19/23/25 — S3 : IO15/16/17/18/48/45. Le role de chaque canal\ndepend du firmware (voir les sections PINMAP_UNIVERSAL). Borniers : 1=NC 2=COM 3=NO.\nSRD Form C = 7A/240VAC et 3A inductif REELS par contact (le 10A ne vaut qu'en 125VAC ou en Form A).\nZONE SECTEUR ISOLEE sur le PCB (fentes + 3mm mini) — circuit 230V\nA PROTEGER EN AMONT (fusible/disjoncteur) ; charges inductives : snubber cote charge." (exclude_from_sim no) (at 271.78 2.54 0)
     (effects (font (size 1.7 1.7)) (justify left bottom)))
-  (text "TOUS les GPIO libres sur header (Dupont),\ny compris RX0/TX0 (les laisser libres pendant le flash USB)\net GPIO36/39 (entrees seules)." (exclude_from_sim no) (at 45.72 162.56 0)
+  (text "HEADER SERVICE J17 : 3V3 / GND / EN / RX0 / TX0 / +5V uniquement.\nTous les autres GPIO sont consommes par la carte universelle\n(GPIO36 = ADC_E, GPIO39 = ADC_VBAT). Laisser RX0/TX0 libres pendant le flash USB." (exclude_from_sim no) (at 45.72 162.56 0)
     (effects (font (size 1.7 1.7)) (justify left bottom)))
   (text "Distribution 5V / 3V3-capteurs / GND :\nborniers a vis + rail header." (exclude_from_sim no) (at 45.72 205.74 0)
