File: hardware/n3-universal/kicad/n3-universal.kicad_sch (KiCad schematic)
At the start: 127 parts, among them J1 Bornier_5.08, J10 JST-XH, J11 Bornier_5.08, J12 Bornier_5.08, J13 Support OLED, J14 Support I2C ext, J15 Header servo, J16 Header servo, J17 Header service, J18 Bornier_5.08, J19 Bornier_5.08, J2 Jack 5.5/2.1, J20 Header alim, J21 Support I2C libre, J22 Support I2C libre, J23 Bornier_5.08, J24 Bornier_5.08, J25 Bornier_5.08, J26 Bornier_5.08, J27 Bornier_5.08, J28 Support I2C libre, J29 JST-XH, J3 Bornier_5.08, J30 JST-XH, J31 Bornier_5.08, J32 Bornier_5.08, J33 Bornier_5.08, J34 Bornier_5.08, J35 Support module microSD, J36 Bornier_5.08, J37 Bornier_5.08, J4 Bornier_5.08, J5 Bornier_5.08, J6 Bornier_5.08, J7 JST-XH, J8 JST-XH, J9 JST-XH, K1 SRD-05VDC-SL-C, K2 SRD-05VDC-SL-C, K3 SRD-05VDC-SL-C, K4 SRD-05VDC-SL-C, K5 SRD-05VDC-SL-C, K6 SRD-05VDC-SL-C, Q1 BC337-40, Q10 BC337-40, Q11 NDP6020P, Q2 BC337-40, Q3 BC337-40, Q4 BC337-40, Q5 BC337-40, Q6 BC337-40, Q7 NDP6020P, Q8 BC337-40, Q9 BS250

Commit message: [n3-universal] rev 0.1.1 : finalisation sous KiCad 10 (DRC 0 erreur, parite schema/PCB)
- plan GND de la bande relais remonte a y86 + regle .kicad_dru mains_vs_gnd_plane
  (ligne de fuite >= 6,5 mm, SEC-CRP-01) ; check_mains_plane_gap couche par couche
- finalize_board.py (retouches idempotentes du PCB route : amorces RV1 2,0 mm,
  serigraphie 0,15 mm, libelles PCB_TEXTS, cartouche, nets NC, trous board-only)
- tidy_silkscreen.py etendu aux libelles ; marquages +/GND, COM = PHASE,
  HC-SR04, UN SEUL MODULE ; labels globaux et fp-lib-table (parite 0 ecart)
- export_fab.py portable Windows (kicad_tools, zipfile, DRC bloquant,
  --subtract-soldermask) ; generate.py ne reecrit plus un PCB route
- gerbers v0.1.1, schema.pdf, SVG, BOM/CPL JLCPCB/NextPCB regeneres ;
  zip v0.1 perime retire ; CPL pcba : rotation J2 ; docs (README, AUDIT §4/§11, COMMANDE)

Co-authored-by: Cursor <cursoragent@cursor.com>
Connections:
- net GND: no longer A1.15 (GPIO23), A2.38 (GPIO48), A2.42 (GPIO19), JP3.3, R28.1
- net I2C_SDA: no longer D7.2 (A), K6.2 (COIL-), LED7.1 (K), Q6.1 (C)
- new net K5: A1.15 (GPIO23), A2.38 (GPIO48), JP3.3, R28.1
- new net REL6_SW: D7.2 (A), K6.2 (COIL-), LED7.1 (K), Q6.1 (C)
Other:
- moved on the sheet: J28, J31, J32, J33, J34, R43, R44, R45, R46
