File: hardware/n3-universal/kicad/n3-universal.kicad_sch (KiCad schematic)
At the start: 172 parts, among them J1 Bornier_5.08, J10 Bornier_5.08, J11 Bornier_5.08, J12 Bornier_5.08, J13 Support OLED, J14 Support I2C ext, J15 Header servo, J16 Header servo, J17 Header service, J18 Bornier_5.08, J19 Bornier_5.08, J2 Jack 5.5/2.1, J20 Header alim, J21 Support I2C libre, J22 Support I2C libre, J23 Bornier_5.08, J24 Bornier_5.08, J25 Bornier_5.08, J26 Bornier_5.08, J27 Bornier_5.08, J28 Support I2C libre, J29 Bornier_5.08, J3 Bornier_5.08, J30 Bornier_5.08, J31 Bornier_5.08, J32 Bornier_5.08, J33 Bornier_5.08, J34 Bornier_5.08, J35 Support module microSD, J36 Bornier_5.08, J37 Bornier_5.08, J38 Header CMD SENSE, J4 Bornier_5.08, J5 Bornier_5.08, J6 Bornier_5.08, J7 Bornier_5.08, J8 Bornier_5.08, J9 Bornier_5.08, K1 SRD-05VDC-SL-C, K2 SRD-05VDC-SL-C, K3 SRD-05VDC-SL-C, K4 SRD-05VDC-SL-C, K5 SRD-05VDC-SL-C, K6 SRD-05VDC-SL-C, Q1 BC337-40, Q11 IRF4905, Q12 IRF4905, Q2 BC337-40, Q3 BC337-40, Q4 BC337-40, Q5 BC337-40, Q6 BC337-40, Q7 IRF4905, Q8 BC337-40, U1 LD1117V33

Commit message: hardware/n3-universal rev 0.2.2 : décisions d'alimentation (servos sur le 5 V commuté, D5 en pont de fil, R39 18k, LED5 par profil), carte reroutée, DRC 0/0/0, gerbers v0.2.2
Suite à ALIMENTATION.md (sobriété et robustesse des quatre profils, commande JLCPCB unique) :
- Servos J15/J16 (pin 2) et C2 passent sur LDO_IN, le 5 V déjà commuté par Q7 : coupés en deep
  sleep sur msp/n3pp (JP1 ôté, -1,2 Wh/j), permanents sur ffp5cs (JP1 fermé). Aucun composant
  ajouté ; une première variante avec un second P-FET (Q13) + cavalier bouchait le couloir de
  pistes du bas de carte (7 nets non routés). SPICE : SG90 bloqué à travers Q7 -> LDO_IN >= 4,91 V,
  +3V3_SW 3,30 V jusqu'à 2,5 A.
- D5 = pont de fil (valeur FIL, empreinte DO-201 conservée) : +0,35 V de marge pour l'AMS1117 du
  DevKit ; règle : ne JAMAIS brancher l'USB du DevKit carte sous tension.
- R39 = 18k (pont VBAT profil 12 V) : 14,5 V mesurés en sortie du PWM -> zone linéaire de l'ADC.
- LED5 non posée sur msp/n3pp (étoilée en BOM).
- Carte reroutée en partant du cuivre validé 0.2.1 comme amorce (un reroutage à blanc laissait
  ADC_D et EN non routés) : freerouting 0 net non routé, secteur/ponts/vias/thermals régénérés,
  check_mains_gap 0, plans GND 6,50 mm. DRC KiCad 10.0.7 avec parité : 0 erreur, 0 non connecté,
  0 écart de parité, 62 avertissements de sérigraphie. Toutes les gardes passent
  (fet_orientation, pinmap_vs_firmware avec J15/J16/C2 sur LDO_IN, silk_refs, pcb_clearance,
  annotate_pcb_roles, sync_pcb_sim_fields, jlcpcb_caps). export_fab --rev 0.2.2 (DRC bloquant
  passé) ; gerbers v0.2.1 retirés.
- ALIMENTATION.md §6 : 14,5 V en sortie du PWM (donnée de terrain) ; §8 décisions ; README,
  COMMANDE.md (10 cartes, v0.2.2), SIMULATION.md, hardware/README.md mis à jour.

Co-Authored-By: Claude Fable 5.1 <noreply@anthropic.com>
Claude-Session: https://claude.ai/code/session_01PiLqx7Upejx4s767q7AD2n
Parts:
- D5: value 1N5822 -> FIL
- R39: value 22k -> 18k
Connections:
- net +5V: no longer C2.1 (+), J15.2, J16.2
- net LDO_IN: now also C2.1 (+), J15.2, J16.2
Other:
- note added: "PONT DIVISEUR VBAT PERMANENT (rev 0.2, plus de coupure BS250) : R38 100k + JP12 : 1-2 = 18k (bus 12V, ffp5cs ; 14,7 V -> 2,24 V) ; 2-3 = 100k (1S Li-ion, msp/n3pp). R49/C13 filtre, D11 clamp 3V3."
- note removed: "PONT DIVISEUR VBAT PERMANENT (rev 0.2, plus de coupure BS250) : R38 100k + JP12 : 1-2 = 22k (bus 12V, ffp5cs) ; 2-3 = 100k (1S Li-ion, msp/n3pp). R49/C13 filtre, D11 clamp 3V3."
